File: wfipic32.brd (EAGLE design)
At the start: 29.2 x 22.5 mm, 8 parts, among them IC1 BMA490L, U1 PIC32MK0512MCJ048T-I/Y8XTQFP4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

Commit message: up
Parts:
- C1, C3, C4, C5: value (none) -> 0.1uf
- C2: value (none) -> 10uf
- L1: value (none) -> 100uh
Changed lines of the file:
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@@
 <attribute name="VALUE" x="10.81" y="40.64" size="1.27" layer="28" rot="MR0" align="center"/>
 </element>
-<element name="C1" library="rcl" library_urn="urn:adsk.eagle:library:334" package="C0805" package3d_urn="urn:adsk.eagle:package:23617/2" value="" x="2.54" y="39.37" smashed="yes" rot="R270">
+<element name="C1" library="rcl" library_urn="urn:adsk.eagle:library:334" package="C0805" package3d_urn="urn:adsk.eagle:package:23617/2" value="0.1uf" x="2.54" y="39.37" smashed="yes" rot="R270">
 <attribute name="NAME" x="3.81" y="40.64" size="1.27" layer="25" rot="R270"/>
 <attribute name="POPULARITY" value="63" x="2.54" y="39.37" size="1.778" layer="27" rot="R270" display="off"/>
@@
 <attribute name="VALUE" x="0" y="40.64" size="1.27" layer="27" rot="R270"/>
 </element>
-<element name="C2" library="rcl" library_urn="urn:adsk.eagle:library:334" package="C0805" package3d_urn="urn:adsk.eagle:package:23617/2" value="" x="3.81" y="33.02" smashed="yes" rot="R180">
+<element name="C2" library="rcl" library_urn="urn:adsk.eagle:library:334" package="C0805" package3d_urn="urn:adsk.eagle:package:23617/2" value="10uf" x="3.81" y="33.02" smashed="yes" rot="R180">
 <attribute name="NAME" x="2.54" y="31.75" size="1.27" layer="25" rot="R180"/>
 <attribute name="POPULARITY" value="63" x="3.81" y="33.02" size="1.778" layer="27" rot="R180" display="off"/>
@@
 <attribute name="VALUE" x="5.08" y="35.56" size="1.27" layer="27" rot="R180"/>
 </element>
-<element name="L1" library="rcl" library_urn="urn:adsk.eagle:library:334" package="L3216C" package3d_urn="urn:adsk.eagle:package:23476/2" value="" x="13.97" y="33.02" smashed="yes">
+<element name="L1" library="rcl" library_urn="urn:adsk.eagle:library:334" package="L3216C" package3d_urn="urn:adsk.eagle:package:23476/2" value="100uh" x="13.97" y="33.02" smashed="yes">
 <attribute name="NAME" x="17.145" y="32.385" size="1.27" layer="25"/>
 <attribute name="POPULARITY" value="3" x="13.97" y="33.02" size="1.778" layer="27" display="off"/>
@@
 <attribute name="VALUE" x="12.065" y="29.845" size="1.27" layer="27"/>
 </element>
-<element name="C3" library="rcl" library_urn="urn:adsk.eagle:library:334" package="C0805" package3d_urn="urn:adsk.eagle:package:23617/2" value="" x="8.89" y="33.02" smashed="yes">
+<element name="C3" library="rcl" library_urn="urn:adsk.eagle:library:334" package="C0805" package3d_urn="urn:adsk.eagle:package:23617/2" value="0.1uf" x="8.89" y="33.02" smashed="yes">
 <attribute name="NAME" x="7.62" y="34.29" size="1.27" layer="25"/>
 <attribute name="POPULARITY" value="63" x="8.89" y="33.02" size="1.778" layer="27" display="off"/>
@@
 <attribute name="VALUE" x="7.62" y="30.48" size="1.27" layer="27"/>
 </element>
-<element name="C4" library="rcl" library_urn="urn:adsk.eagle:library:334" package="C0805" package3d_urn="urn:adsk.eagle:package:23617/2" value="" x="10.16" y="43.18" smashed="yes" rot="MR180">
+<element name="C4" library="rcl" library_urn="urn:adsk.eagle:library:334" package="C0805" package3d_urn="urn:adsk.eagle:package:23617/2" value="0.1uf" x="10.16" y="43.18" smashed="yes" rot="MR180">
 <attribute name="NAME" x="8.89" y="41.91" size="1.27" layer="26" rot="MR180"/>
 <attribute name="POPULARITY" value="63" x="10.16" y="43.18" size="1.778" layer="28" rot="MR180" display="off"/>
@@
 <attribute name="VALUE" x="8.89" y="45.72" size="1.27" layer="28" rot="MR180"/>
 </element>
-<element name="C5" library="rcl" library_urn="urn:adsk.eagle:library:334" package="C0805" package3d_urn="urn:adsk.eagle:package:23617/2" value="" x="10.16" y="38.1" smashed="yes" rot="MR0">
+<element name="C5" library="rcl" library_urn="urn:adsk.eagle:library:334" package="C0805" package3d_urn="urn:adsk.eagle:package:23617/2" value="0.1uf" x="10.16" y="38.1" smashed="yes" rot="MR0">
 <attribute name="NAME" x="11.43" y="39.37" size="1.27" layer="26" rot="MR0"/>
 <attribute name="POPULARITY" value="63" x="10.16" y="38.1" size="1.778" layer="28" rot="MR0" display="off"/>

Commit message: up
Parts:
- added C6: 0.1uf, rcl:C0805
- added C7: 10uf, rcl:C0805
- added J1, J2: MLE-105-01-G-DV, MLE-105-01-G-DV:MLE-105-01-G-DV
- added JP1: RESET_JMP, pinhead:1X02
- added JP2: ICSP, pinhead:1X06
- added LED1: RED, led:CHIPLED_0603
- added LED2: GREEN, led:CHIPLED_0603
- added R1, R2, R3, R4: 2k, rcl:M0805
Connections:
- new net EXT_INT2: IC1.5, U1.35
- new net GREEN_LED: R2.2, U1.27
- new net IMU_CS: IC1.10, U1.41
- new net MCLR_SIG: JP2.1, R4.2, U1.4
- new net N$1: LED1.A, R1.1
- new net N$2: LED2.A, R2.1
- new net N$3: C6.1, JP1.1, R3.1, R4.1
- new net PGC: JP2.5, U1.13
- new net PGD: JP2.4, U1.14
- new net RED_LED: R1.2, U1.28
- new net SCK2: IC1.12, U1.38
- new net SDI2: IC1.1, U1.40
- new net SDO2: IC1.2, U1.39
- new net U1RX: J1.2, U1.18
- new net U1TX: J1.3, U1.19
- net VDD: now also C7.1, J1.10, J2.10, JP2.2, R3.2
- net VSS: now also C6.2, C7.2, J1.1, J2.1, JP1.2, JP2.3, LED1.C, LED2.C
Routing:
- net VSS: track 62.3 -> 176.3 mm, vias 1 -> 2
- net VDD: track 41.9 -> 112.5 mm, vias 1 -> 3
- net N$3: track 0.00 -> 41.7 mm
- net MCLR_SIG: track 0.00 -> 38.8 mm
- net PGD: track 0.00 -> 35.8 mm
- net PGC: track 0.00 -> 28.9 mm, vias 0 -> 1
- net U1RX: track 0.00 -> 15.6 mm
- net RED_LED: track 0.00 -> 14.2 mm
- net U1TX: track 0.00 -> 13.5 mm, vias 0 -> 2
- net GREEN_LED: track 0.00 -> 13.2 mm
- net N$2: track 0.00 -> 12.0 mm
- net SDO2: track 0.00 -> 11.1 mm, vias 0 -> 1
- net EXT_INT2: track 0.00 -> 10.4 mm, vias 0 -> 2
- net SDI2: track 0.00 -> 9.66 mm, vias 0 -> 1
- net SCK2: track 0.00 -> 5.41 mm, vias 0 -> 1
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- added copper zone on layer 2, net VSS
Other:
- board size 29.2 x 22.5 mm -> 31.7 x 25.1 mm

Commit message: up
Parts:
- added J3: MLE-105-01-G-DV, MLE-105-01-G-DV:MLE-105-01-G-DV
- moved JP1 10.2 mm to (11.4, 50.8), turned to 90 degrees
- moved R2 7.73 mm to (7.62, 49.5)
- moved R1 2.84 mm to (7.62, 52.1)
- moved LED1 2.54 mm to (3.81, 50.8)
- moved LED2 1.80 mm to (3.81, 52.1)
Connections:
- new net AN0: J2.3, U1.9
- new net AN1: J2.5, U1.10
- new net DAC1: J2.9, U1.33
- new net EXT_SW1: J1.6, U1.8
- new net EXT_SW2: J1.8, U1.7
- new net INDX2: J2.6, U1.46
- new net QEA2: J2.2, U1.45
- new net QEB2: J2.4, U1.47
- new net SDI1: J1.5, U1.24
- new net SDI1_MODE: J1.4, U1.37
- new net SDO1: J1.7, U1.31
- new net SS1_OUT: J1.9, U1.32
- new net VREF+: J2.7, U1.12
- net VSS: now also J3.1
Routing:
- net VSS: track 176.3 -> 99.1 mm, vias 2 -> 3
- net AN1: track 0.00 -> 26.2 mm, vias 0 -> 2
- net N$3: track 41.7 -> 15.9 mm
- net SS1_OUT: track 0.00 -> 24.4 mm, vias 0 -> 2
- net QEA2: track 0.00 -> 23.1 mm, vias 0 -> 2
- net AN0: track 0.00 -> 20.2 mm, vias 0 -> 2
- net SDO1: track 0.00 -> 18.6 mm, vias 0 -> 2
- net QEB2: track 0.00 -> 17.2 mm
- net EXT_SW2: track 0.00 -> 16.6 mm
- net EXT_SW1: track 0.00 -> 16.5 mm, vias 0 -> 2
- net VREF+: track 0.00 -> 16.0 mm, vias 0 -> 2
- net INDX2: track 0.00 -> 15.5 mm
- net SDI1_MODE: track 0.00 -> 14.1 mm
- net SDI1: track 0.00 -> 9.34 mm
- net PGC: track 28.9 -> 38.2 mm
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
Commit message: up
Parts:
- moved C4 2.54 mm to (7.62, 43.2)
- moved C5 2.54 mm to (7.62, 38.1)
Connections:
- new net PWM1H: J3.9, U1.2
- new net PWM1L: J3.7, U1.3
- new net PWM4H: J3.10, U1.48
- new net PWM4L: J3.8, U1.1
- net VSS: now also J3.2
Routing:
- net PWM1L: track 0.00 -> 21.2 mm, vias 0 -> 2
- net PWM4L: track 0.00 -> 20.9 mm, vias 0 -> 2
- net VSS: track 99.1 -> 114.6 mm, vias 3 -> 4
- net PWM1H: track 0.00 -> 15.1 mm, vias 0 -> 2
- net PWM4H: track 0.00 -> 14.0 mm
- net EXT_SW1: track 16.5 -> 28.8 mm
- net SS1_OUT: track 24.4 -> 12.3 mm
- net SDI2: track 19.0 -> 7.44 mm
- net MCLR_SIG: track 36.4 -> 25.9 mm, vias 2 -> 1
- net AN1: track 26.2 -> 36.1 mm
- net EXT_INT2: track 11.4 -> 20.9 mm, vias 2 -> 1
- net IMU_CS: track 12.8 -> 3.56 mm, vias 2 -> 1
- net VREF+: track 16.0 -> 24.0 mm
- net QEB2: track 17.2 -> 23.4 mm
- net VDD: track 111.8 -> 105.6 mm, vias 1 -> 4
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
Commit message: up
Parts:
- added C10, C8, C9: 0.1uf, rcl:C0805
- added C11: 10uf, rcl:C0805
- added REFCLK2, TP1, TP2, TP3: PTR1PAD1-13, testpad:P1-13
- added U2: MAX6126B30, MAX6126B30:SOP65P490X110-8N
- moved JP2 2.84 mm to (27.9, 40.6)
- moved C2 1.27 mm to (3.81, 31.8)
- moved C3 1.27 mm to (8.89, 31.8)
- moved C7 1.27 mm to (26.7, 31.8)
- moved L1 1.27 mm to (14.0, 31.8)
Connections:
- new net N$4: C8.1, U2.1
- new net N$5: TP1.TP, U1.20
- new net N$6: TP2.TP, U1.19
- new net N$7: TP3.TP, U1.11
- new net N$8: REFCLK2.TP, U1.25
- new net PWM1EN: J3.5, U1.30
- new net PWM1ER: J3.3, U1.36
- new net PWM4EN: J3.6, U1.45
- new net PWM4ER: J3.4, U1.23
- new net SCK1: J1.8, U1.34
- net AVDD: now also C10.1, U2.2
- net EXT_SW2: now also J2.8; no longer J1.8
- net QEA2: now also U1.44; no longer U1.45
- net U1TX: now also U1.17; no longer U1.19
- net VREF+: now also C11.1, C9.1, U2.6, U2.7
- net VSS: now also C10.2, C11.2, C8.2, C9.2, U2.3, U2.4
Routing:
- net PWM4ER: track 0.00 -> 52.0 mm, vias 0 -> 2
- net N$5: track 0.00 -> 50.3 mm, vias 0 -> 1
- net VSS: track 114.6 -> 151.7 mm, vias 4 -> 3
- net N$7: track 0.00 -> 33.4 mm, vias 0 -> 2
- net U1TX: track 13.8 -> 33.3 mm
- net PWM4EN: track 0.00 -> 19.3 mm, vias 0 -> 2
- net PWM1EN: track 0.00 -> 16.5 mm, vias 0 -> 2
- net VREF+: track 24.0 -> 40.2 mm, vias 2 -> 3
- net AVDD: track 8.41 -> 23.9 mm, vias 0 -> 2
- net SCK1: track 0.00 -> 14.0 mm, vias 0 -> 2
- net AN1: track 36.1 -> 22.4 mm
- net EXT_SW2: track 16.6 -> 26.2 mm, vias 0 -> 2
- net PWM1ER: track 0.00 -> 9.09 mm
- net VDD: track 105.6 -> 114.4 mm
- net QEB2: track 23.4 -> 16.9 mm, vias 0 -> 2
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Other:
- board size 31.7 x 25.1 mm -> 33 x 25.1 mm

Commit message: up
Parts:
- R3: value 2k -> 10k
- R4: value 2k -> 56
- moved JP2 2.84 mm to (29.2, 43.2)
- moved JP1 1.80 mm to (12.7, 52.1), turned to 180 degrees
- moved TP1 1.27 mm to (25.4, 43.2)
- moved TP2 1.27 mm to (25.4, 40.6)
- moved TP3 1.27 mm to (25.4, 38.1)
Connections:
- removed net N$7: TP3.TP, U1.11
- new net BMA_INT2: IC1.6, TP3.TP, U1.11
Routing:
- net BMA_INT2: track 0.00 -> 42.9 mm, vias 0 -> 1
- net N$7: track 33.4 -> 0.00 mm, vias 2 -> 0
- net N$5: track 50.3 -> 19.1 mm
- net GREEN_LED: track 14.3 -> 43.2 mm
- net N$6: track 0.00 -> 27.7 mm
- net PWM4ER: track 52.0 -> 25.1 mm
- net VSS: track 151.7 -> 130.7 mm, vias 3 -> 4
- net PGD: track 26.7 -> 44.6 mm, vias 1 -> 0
- net MCLR_SIG: track 29.9 -> 47.6 mm
- net U1TX: track 33.3 -> 18.4 mm
- net QEB2: track 16.9 -> 27.5 mm
- net SDI1_MODE: track 15.8 -> 25.9 mm
- net EXT_SW1: track 28.1 -> 19.3 mm
- net EXT_INT2: track 19.2 -> 11.5 mm, vias 2 -> 1
- net PWM1L: track 16.5 -> 23.9 mm, vias 2 -> 0
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Other:
- board size 33 x 25.1 mm -> 35.5 x 27.6 mm
- board text added: "BMA490L-PIC32MK V1.0"

Commit message: up
Parts:
- moved C1 2.54 mm to (2.54, 36.8)
- moved C4 1.27 mm to (7.62, 44.5)
- moved C5 1.27 mm to (7.62, 36.8)
Routing:
- net GREEN_LED: track 43.2 -> 18.4 mm
- net VDD: track 114.5 -> 135.0 mm
- net EXT_SW2: track 21.5 -> 38.5 mm
- net PWM4ER: track 25.1 -> 39.4 mm
- net PWM1EN: track 23.6 -> 11.1 mm, vias 0 -> 2
- net VSS: track 130.7 -> 141.0 mm, vias 4 -> 2
- net PWM1ER: track 9.07 -> 19.0 mm, vias 0 -> 2
- net PGC: track 33.4 -> 42.5 mm
- net SS1_OUT: track 21.7 -> 12.9 mm
- net MCLR_SIG: track 47.6 -> 38.9 mm, vias 1 -> 3
- net N$6: track 27.7 -> 20.6 mm, vias 0 -> 2
- net N$3: track 22.8 -> 29.5 mm, vias 0 -> 1
- net SDI1_MODE: track 25.9 -> 20.4 mm
- net SCK1: track 16.1 -> 10.8 mm
- net VREF+: track 47.1 -> 41.8 mm
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