File: wfipic32.sch (EAGLE design)
At the start: 8 parts, among them IC1 BMA490L, U1 PIC32MK0512MCJ048T-I/Y8XTQFP4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

Commit message: up
Parts:
- C1, C3, C4, C5: value (none) -> 0.1uf
- C2: value (none) -> 10uf
- L1: value (none) -> 100uh
Changed lines of the file:
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@@
 <part name="U1" library="2022-08-07_22-50-41_Library" deviceset="PIC32MK0512MCJ048T-I/Y8X" device="TQFP48_Y8X_MCH-M"/>
 <part name="IC1" library="SamacSys_Parts" deviceset="BMA490L" device=""/>
-<part name="C1" library="rcl" library_urn="urn:adsk.eagle:library:334" deviceset="C-US" device="C0805" package3d_urn="urn:adsk.eagle:package:23617/2"/>
-<part name="C2" library="rcl" library_urn="urn:adsk.eagle:library:334" deviceset="C-US" device="C0805" package3d_urn="urn:adsk.eagle:package:23617/2"/>
+<part name="C1" library="rcl" library_urn="urn:adsk.eagle:library:334" deviceset="C-US" device="C0805" package3d_urn="urn:adsk.eagle:package:23617/2" value="0.1uf"/>
+<part name="C2" library="rcl" library_urn="urn:adsk.eagle:library:334" deviceset="C-US" device="C0805" package3d_urn="urn:adsk.eagle:package:23617/2" value="10uf"/>
 <part name="VDD1" library="supply1" library_urn="urn:adsk.eagle:library:371" deviceset="VDD" device=""/>
 <part name="VSS1" library="supply1" library_urn="urn:adsk.eagle:library:371" deviceset="VSS" device=""/>
-<part name="L1" library="rcl" library_urn="urn:adsk.eagle:library:334" deviceset="L-US" device="L3216C" package3d_urn="urn:adsk.eagle:package:23476/2"/>
-<part name="C3" library="rcl" library_urn="urn:adsk.eagle:library:334" deviceset="C-US" device="C0805" package3d_urn="urn:adsk.eagle:package:23617/2"/>
+<part name="L1" library="rcl" library_urn="urn:adsk.eagle:library:334" deviceset="L-US" device="L3216C" package3d_urn="urn:adsk.eagle:package:23476/2" value="100uh"/>
+<part name="C3" library="rcl" library_urn="urn:adsk.eagle:library:334" deviceset="C-US" device="C0805" package3d_urn="urn:adsk.eagle:package:23617/2" value="0.1uf"/>
 <part name="VSS2" library="supply1" library_urn="urn:adsk.eagle:library:371" deviceset="VSS" device=""/>
-<part name="C4" library="rcl" library_urn="urn:adsk.eagle:library:334" deviceset="C-US" device="C0805" package3d_urn="urn:adsk.eagle:package:23617/2"/>
-<part name="C5" library="rcl" library_urn="urn:adsk.eagle:library:334" deviceset="C-US" device="C0805" package3d_urn="urn:adsk.eagle:package:23617/2"/>
+<part name="C4" library="rcl" library_urn="urn:adsk.eagle:library:334" deviceset="C-US" device="C0805" package3d_urn="urn:adsk.eagle:package:23617/2" value="0.1uf"/>
+<part name="C5" library="rcl" library_urn="urn:adsk.eagle:library:334" deviceset="C-US" device="C0805" package3d_urn="urn:adsk.eagle:package:23617/2" value="0.1uf"/>
 <part name="VSS3" library="supply1" library_urn="urn:adsk.eagle:library:371" deviceset="VSS" device=""/>
 <part name="VSS4" library="supply1" library_urn="urn:adsk.eagle:library:371" deviceset="VSS" device=""/>
@@
 <pinref part="VDD1" gate="G$1" pin="VDD"/>
 <pinref part="L1" gate="G$1" pin="2"/>
+<junction x="5.08" y="132.08"/>
 </segment>
 <segment>
@@
 <junction x="99.06" y="132.08"/>
 <pinref part="C5" gate="G$1" pin="1"/>
+<junction x="99.06" y="144.78"/>
 </segment>
 <segment>
@@
 <junction x="96.52" y="93.98"/>
 <pinref part="C4" gate="G$1" pin="1"/>
+<junction x="96.52" y="83.82"/>
 </segment>
 <segment>
 <wire x1="200.66" y1="58.42" x2="213.36" y2="58.42" width="0.1524" layer="91"/>
 <pinref part="U1" gate="A" pin="VDD"/>
+<junction x="200.66" y="58.42"/>
+<junction x="213.36" y="58.42"/>
+<label x="205.74" y="58.42" size="1.778" layer="95"/>
 </segment>
 <segment>
 <wire x1="-30.48" y1="58.42" x2="-17.78" y2="58.42" width="0.1524" layer="91"/>
 <pinref part="U1" gate="A" pin="VDD_2"/>
+<junction x="-17.78" y="58.42"/>
+<junction x="-30.48" y="58.42"/>
+<label x="-27.94" y="58.42" size="1.778" layer="95"/>
 </segment>
 <segment>
 <wire x1="-30.48" y1="17.78" x2="-17.78" y2="17.78" width="0.1524" layer="91"/>
 <pinref part="U1" gate="A" pin="VDD_3"/>
+<junction x="-17.78" y="17.78"/>
+<junction x="-30.48" y="17.78"/>
+<label x="-27.94" y="17.78" size="1.778" layer="95"/>
 </segment>
 <segment>
 <wire x1="200.66" y1="15.24" x2="213.36" y2="15.24" width="0.1524" layer="91"/>
 <pinref part="U1" gate="A" pin="VDD_4"/>
+<junction x="200.66" y="15.24"/>
+<junction x="213.36" y="15.24"/>
+<label x="205.74" y="15.24" size="1.778" layer="95"/>
 </segment>
 </net>
@@
 <label x="27.94" y="121.92" size="1.778" layer="95"/>
 <pinref part="VSS1" gate="G$1" pin="VSS"/>
+<junction x="5.08" y="124.46"/>
 </segment>
 <segment>
@@
 <pinref part="IC1" gate="G$1" pin="GND"/>
 <junction x="93.98" y="132.08"/>
+<junction x="93.98" y="144.78"/>
 </segment>
 <segment>
@@
 <pinref part="IC1" gate="G$1" pin="GNDIO"/>
 <junction x="96.52" y="132.08"/>
+<junction x="96.52" y="144.78"/>
 </segment>
 <segment>
 <wire x1="-30.48" y1="60.96" x2="-17.78" y2="60.96" width="0.1524" layer="91"/>
 <pinref part="U1" gate="A" pin="VSS_2"/>
+<junction x="-17.78" y="60.96"/>
+<junction x="-30.48" y="60.96"/>
+<label x="-27.94" y="60.96" size="1.778" layer="95"/>
 </segment>
 <segment>
 <wire x1="-30.48" y1="20.32" x2="-17.78" y2="20.32" width="0.1524" layer="91"/>
 <pinref part="U1" gate="A" pin="VSS_3"/>
+<junction x="-17.78" y="20.32"/>
+<junction x="-30.48" y="20.32"/>
+<label x="-27.94" y="20.32" size="1.778" layer="95"/>
 </segment>
 <segment>
 <wire x1="200.66" y1="55.88" x2="213.36" y2="55.88" width="0.1524" layer="91"/>
 <pinref part="U1" gate="A" pin="VSS"/>
+<junction x="200.66" y="55.88"/>
+<junction x="213.36" y="55.88"/>
+<label x="208.28" y="55.88" size="1.778" layer="95"/>
 </segment>
 <segment>
 <wire x1="200.66" y1="22.86" x2="213.36" y2="22.86" width="0.1524" layer="91"/>
 <pinref part="U1" gate="A" pin="VSS_4"/>
-</segment>
-<segment>
-<wire x1="-30.48" y1="33.02" x2="-17.78" y2="33.02" width="0.1524" layer="91"/>
+<junction x="200.66" y="22.86"/>
+<junction x="213.36" y="22.86"/>
+<label x="205.74" y="22.86" size="1.778" layer="95"/>
+</segment>
+<segment>
+<wire x1="-30.48" y1="33.02" x2="-27.94" y2="33.02" width="0.1524" layer="91"/>
 <pinref part="U1" gate="A" pin="AVSS"/>
+<junction x="-17.78" y="33.02"/>
+<junction x="-27.94" y="33.02"/>
+<wire x1="-27.94" y1="33.02" x2="-17.78" y2="33.02" width="0.1524" layer="91"/>
+<junction x="-30.48" y="33.02"/>
+<label x="-25.4" y="33.02" size="1.778" layer="95"/>
 </segment>
 <segment>
@@
 <pinref part="C4" gate="G$1" pin="2"/>
 <pinref part="VSS3" gate="G$1" pin="VSS"/>
+<junction x="104.14" y="83.82"/>
 </segment>
 <segment>
 <pinref part="C5" gate="G$1" pin="2"/>
 <pinref part="VSS4" gate="G$1" pin="VSS"/>
+<junction x="106.68" y="144.78"/>
 </segment>
 </net>
@@
 <wire x1="-25.4" y1="35.56" x2="-17.78" y2="35.56" width="0.1524" layer="91"/>
 <pinref part="U1" gate="A" pin="AVDD"/>
+<junction x="-17.78" y="35.56"/>
+<junction x="-25.4" y="35.56"/>
+<label x="-22.86" y="35.56" size="1.778" layer="95"/>
 </segment>
 </net>

Commit message: up
Parts:
- added C6: 0.1uf, rcl:C-USC0805
- added C7: 10uf, rcl:C-USC0805
- added J1, J2: MLE-105-01-G-DV, MLE-105-01-G-DV:MLE-105-01-G-DV
- added JP1: RESET_JMP, pinhead:PINHD-1X2
- added JP2: ICSP, pinhead:PINHD-1X6
- added LED1: RED, led:LEDCHIPLED_0603
- added LED2: GREEN, led:LEDCHIPLED_0603
- added R1, R2, R3, R4: 2k, rcl:R-US_M0805
Connections:
- new net EXT_INT2: IC1.INT1, U1.SOSCI/RPC13/RC13
- new net GREEN_LED: R2.2, U1.OSCI/CLKI/AN49/CVD49/RPC12/RC12
- new net IMU_CS: IC1.CSB, U1.RPC9/PWM5L/RC9
- new net MCLR_SIG: JP2.1, R4.2, U1.MCLR
- new net N$1: LED1.A, R1.1
- new net N$2: LED2.A, R2.1
- new net N$3: C6.1, JP1.1, R3.1, R4.1
- new net PGC: JP2.5, U1.PGC1/OA1IN+/AN4/C1IN1+/C1IN3-/C2IN3-/RPB2/RB2
- new net PGD: JP2.4, U1.PGD1/OA1IN-/AN5/CTCMP/C1IN1-/RTCC/RPB3/RB3
- new net RED_LED: R1.2, U1.OSCO/CLKO/RPC15/RC15
- new net SCK2: IC1.SCX, U1.RPC6/PWM6H/RC6
- new net SDI2: IC1.SDO, U1.RPC8/PWM5H/RC8
- new net SDO2: IC1.SDX, U1.RPC7/PWM6L/RC7
- new net U1RX: J1.2, U1.OA3IN-/AN7/CVD7/C3IN1-/C4IN1-/RPC1/RC1
- new net U1TX: J1.3, U1.OA3IN+/AN8/CVD8/C3IN1+/C3IN3-/RPC2/FLT3/RC2
- net VDD: now also C7.1, J1.10, J2.10, JP2.2, R3.2
- net VSS: now also C6.2, C7.2, J1.1, J2.1, JP1.2, JP2.3, LED1.C, LED2.C

Commit message: up
Parts:
- added J3: MLE-105-01-G-DV, MLE-105-01-G-DV:MLE-105-01-G-DV
Connections:
- new net AN0: J2.3, U1.OA2OUT/AN0/C2IN4-/C4IN3-/RPA0/RA0
- new net AN1: J2.5, U1.OA2IN+/AN1/C2IN1+/RPA1/RA1
- new net DAC1: J2.9, U1.DAC1/AN48/CVD48/RPC10/RC10
- new net EXT_SW1: J1.6, U1.AN9/CVD9/RPA11/FLT14/RA11
- new net EXT_SW2: J1.8, U1.AN10/CVD10/RPA12/FLT13/RA12
- new net INDX2: J2.6, U1.RPB12/PWM2H/RB12
- new net QEA2: J2.2, U1.RPB11/PWM3L/RB11
- new net QEB2: J2.4, U1.RPB13/PWM2L/CTPLS/RB13
- new net SDI1: J1.5, U1.FLT15/RPB4/SCL2/RB4
- new net SDI1_MODE: J1.4, U1.TMS/OA5IN-/AN27/CVD27/LVDIN/C5IN1-/RPB9/RB9
- new net SDO1: J1.7, U1.PGD2/RPB5/SDA1/RB5
- new net SS1_OUT: J1.9, U1.PGC2/RPB6/SCL1/RB6
- new net VREF+: J2.7, U1.PGC3/OA1OUT/VREF+/AN3/C1IN4-/C4IN2-/RPB1/CTED1/RB1
- net VSS: now also J3.1
Changed lines of the file:
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@@
 <part name="C7" library="rcl" library_urn="urn:adsk.eagle:library:334" deviceset="C-US" device="C0805" package3d_urn="urn:adsk.eagle:package:23617/2" value="10uf"/>
 <part name="VSS12" library="supply1" library_urn="urn:adsk.eagle:library:371" deviceset="VSS" device=""/>
+<part name="J3" library="MLE-105-01-G-DV" deviceset="MLE-105-01-G-DV" device=""/>
+<part name="VSS13" library="supply1" library_urn="urn:adsk.eagle:library:371" deviceset="VSS" device=""/>
 </parts>
 <sheets>
@@
 <instance part="VSS12" gate="G$1" x="213.36" y="83.82" smashed="yes">
 <attribute name="VALUE" x="210.82" y="78.74" size="1.778" layer="96" rot="R90"/>
+</instance>
+<instance part="J3" gate="G$1" x="170.18" y="-5.08" smashed="yes">
+<attribute name="NAME" x="189.23" y="2.54" size="1.778" layer="95" align="center-left"/>
+<attribute name="VALUE" x="189.23" y="0" size="1.778" layer="96" align="center-left"/>
+</instance>
+<instance part="VSS13" gate="G$1" x="170.18" y="-17.78" smashed="yes">
+<attribute name="VALUE" x="167.64" y="-22.86" size="1.778" layer="96" rot="R90"/>
 </instance>
 </instances>
@@
 <junction x="213.36" y="86.36"/>
 </segment>
+<segment>
+<pinref part="J3" gate="G$1" pin="1"/>
+<pinref part="VSS13" gate="G$1" pin="VSS"/>
+<junction x="170.18" y="-15.24"/>
+</segment>
 </net>
 <net name="AVDD" class="0">
@@
 </segment>
 </net>
+<net name="SDI1_MODE" class="0">
+<segment>
+<pinref part="U1" gate="A" pin="TMS/OA5IN-/AN27/CVD27/LVDIN/C5IN1-/RPB9/RB9"/>
+<wire x1="200.66" y1="43.18" x2="213.36" y2="43.18" width="0.1524" layer="91"/>
+<label x="215.9" y="43.18" size="1.778" layer="95"/>
+<junction x="200.66" y="43.18"/>
+<junction x="213.36" y="43.18"/>
+</segment>
+<segment>
+<wire x1="193.04" y1="121.92" x2="205.74" y2="121.92" width="0.1524" layer="91"/>
+<pinref part="J1" gate="G$1" pin="4"/>
+<label x="208.28" y="121.92" size="1.778" layer="95"/>
+<junction x="193.04" y="121.92"/>
+<junction x="205.74" y="121.92"/>
+</segment>
+</net>
+<net name="SDI1" class="0">
+<segment>
+<pinref part="U1" gate="A" pin="FLT15/RPB4/SCL2/RB4"/>
+<wire x1="-17.78" y1="12.7" x2="-30.48" y2="12.7" width="0.1524" layer="91"/>
+<label x="-38.1" y="12.7" size="1.778" layer="95"/>
+<junction x="-30.48" y="12.7"/>
+<junction x="-17.78" y="12.7"/>
+</segment>
+<segment>
+<wire x1="170.18" y1="124.46" x2="157.48" y2="124.46" width="0.1524" layer="91"/>
+<pinref part="J1" gate="G$1" pin="5"/>
+<junction x="170.18" y="124.46"/>
+<junction x="157.48" y="124.46"/>
+<label x="147.32" y="124.46" size="1.778" layer="95"/>
+</segment>
+</net>
+<net name="SDO1" class="0">
+<segment>
+<pinref part="U1" gate="A" pin="PGD2/RPB5/SDA1/RB5"/>
+<wire x1="200.66" y1="27.94" x2="213.36" y2="27.94" width="0.1524" layer="91"/>
+<label x="215.9" y="27.94" size="1.778" layer="95"/>
+<junction x="200.66" y="27.94"/>
+<junction x="213.36" y="27.94"/>
+</segment>
+<segment>
+<wire x1="157.48" y1="127" x2="170.18" y2="127" width="0.1524" layer="91"/>
+<pinref part="J1" gate="G$1" pin="7"/>
+<label x="147.32" y="127" size="1.778" layer="95"/>
+<junction x="157.48" y="127"/>
+<junction x="170.18" y="127"/>
+</segment>
+</net>
+<net name="SS1_OUT" class="0">
+<segment>
+<pinref part="U1" gate="A" pin="PGC2/RPB6/SCL1/RB6"/>
+<wire x1="200.66" y1="30.48" x2="213.36" y2="30.48" width="0.1524" layer="91"/>
+<label x="215.9" y="30.48" size="1.778" layer="95"/>
+<junction x="200.66" y="30.48"/>
+<junction x="213.36" y="30.48"/>
+</segment>
+<segment>
+<wire x1="157.48" y1="129.54" x2="170.18" y2="129.54" width="0.1524" layer="91"/>
+<pinref part="J1" gate="G$1" pin="9"/>
+<label x="142.24" y="129.54" size="1.778" layer="95"/>
+<junction x="170.18" y="129.54"/>
+<junction x="157.48" y="129.54"/>
+</segment>
+</net>
+<net name="EXT_SW1" class="0">
+<segment>
+<pinref part="U1" gate="A" pin="AN9/CVD9/RPA11/FLT14/RA11"/>
+<wire x1="-17.78" y1="53.34" x2="-30.48" y2="53.34" width="0.1524" layer="91"/>
+<label x="-40.64" y="53.34" size="1.778" layer="95"/>
+<junction x="-17.78" y="53.34"/>
+<junction x="-30.48" y="53.34"/>
+</segment>
+<segment>
+<wire x1="205.74" y1="124.46" x2="193.04" y2="124.46" width="0.1524" layer="91"/>
+<pinref part="J1" gate="G$1" pin="6"/>
+<label x="208.28" y="124.46" size="1.778" layer="95"/>
+<junction x="193.04" y="124.46"/>
+<junction x="205.74" y="124.46"/>
+</segment>
+</net>
+<net name="EXT_SW2" class="0">
+<segment>
+<pinref part="U1" gate="A" pin="AN10/CVD10/RPA12/FLT13/RA12"/>
+<wire x1="-17.78" y1="55.88" x2="-30.48" y2="55.88" width="0.1524" layer="91"/>
+<label x="-40.64" y="55.88" size="1.778" layer="95"/>
+<junction x="-17.78" y="55.88"/>
+<junction x="-30.48" y="55.88"/>
+</segment>
+<segment>
+<wire x1="205.74" y1="127" x2="193.04" y2="127" width="0.1524" layer="91"/>
+<pinref part="J1" gate="G$1" pin="8"/>
+<label x="208.28" y="127" size="1.778" layer="95"/>
+<junction x="193.04" y="127"/>
+<junction x="205.74" y="127"/>
+</segment>
+</net>
+<net name="AN0" class="0">
+<segment>
+<pinref part="U1" gate="A" pin="OA2OUT/AN0/C2IN4-/C4IN3-/RPA0/RA0"/>
+<wire x1="-17.78" y1="50.8" x2="-30.48" y2="50.8" width="0.1524" layer="91"/>
+<label x="-40.64" y="50.8" size="1.778" layer="95"/>
+<junction x="-17.78" y="50.8"/>
+<junction x="-30.48" y="50.8"/>
+</segment>
+<segment>
+<wire x1="170.18" y1="86.36" x2="157.48" y2="86.36" width="0.1524" layer="91"/>
+<pinref part="J2" gate="G$1" pin="3"/>
+<label x="147.32" y="86.36" size="1.778" layer="95"/>
+<junction x="170.18" y="86.36"/>
+<junction x="157.48" y="86.36"/>
+</segment>
+</net>
+<net name="AN1" class="0">
+<segment>
+<pinref part="U1" gate="A" pin="OA2IN+/AN1/C2IN1+/RPA1/RA1"/>
+<wire x1="-17.78" y1="48.26" x2="-30.48" y2="48.26" width="0.1524" layer="91"/>
+<label x="-40.64" y="48.26" size="1.778" layer="95"/>
+<junction x="-17.78" y="48.26"/>
+<junction x="-30.48" y="48.26"/>
+</segment>
+<segment>
+<wire x1="170.18" y1="88.9" x2="157.48" y2="88.9" width="0.1524" layer="91"/>
+<pinref part="J2" gate="G$1" pin="5"/>
+<label x="147.32" y="88.9" size="1.778" layer="95"/>
+<junction x="170.18" y="88.9"/>
+<junction x="157.48" y="88.9"/>
+</segment>
+</net>
+<net name="VREF+" class="0">
+<segment>
+<pinref part="U1" gate="A" pin="PGC3/OA1OUT/VREF+/AN3/C1IN4-/C4IN2-/RPB1/CTED1/RB1"/>
+<wire x1="-17.78" y1="43.18" x2="-30.48" y2="43.18" width="0.1524" layer="91"/>
+<label x="-43.18" y="43.18" size="1.778" layer="95"/>
+<junction x="-17.78" y="43.18"/>
+<junction x="-30.48" y="43.18"/>
+</segment>
+<segment>
+<wire x1="170.18" y1="91.44" x2="157.48" y2="91.44" width="0.1524" layer="91"/>
+<pinref part="J2" gate="G$1" pin="7"/>
+<label x="147.32" y="91.44" size="1.778" layer="95"/>
+<junction x="170.18" y="91.44"/>
+<junction x="157.48" y="91.44"/>
+</segment>
+</net>
+<net name="DAC1" class="0">
+<segment>
+<pinref part="U1" gate="A" pin="DAC1/AN48/CVD48/RPC10/RC10"/>
+<wire x1="200.66" y1="33.02" x2="213.36" y2="33.02" width="0.1524" layer="91"/>
+<label x="215.9" y="33.02" size="1.778" layer="95"/>
+<junction x="200.66" y="33.02"/>
+<junction x="213.36" y="33.02"/>
+</segment>
+<segment>
+<wire x1="157.48" y1="93.98" x2="170.18" y2="93.98" width="0.1524" layer="91"/>
+<pinref part="J2" gate="G$1" pin="9"/>
+<junction x="170.18" y="93.98"/>
+<junction x="157.48" y="93.98"/>
+<label x="147.32" y="93.98" size="1.778" layer="95"/>
+</segment>
+</net>
+<net name="QEA2" class="0">
+<segment>
+<pinref part="U1" gate="A" pin="RPB11/PWM3L/RB11"/>
+<wire x1="200.66" y1="63.5" x2="213.36" y2="63.5" width="0.1524" layer="91"/>
+<label x="215.9" y="63.5" size="1.778" layer="95"/>
+<junction x="200.66" y="63.5"/>
+<junction x="213.36" y="63.5"/>
+</segment>
+<segment>
+<wire x1="193.04" y1="83.82" x2="205.74" y2="83.82" width="0.1524" layer="91"/>
+<pinref part="J2" gate="G$1" pin="2"/>
+<label x="198.12" y="81.28" size="1.778" layer="95"/>
+<junction x="193.04" y="83.82"/>
+<junction x="205.74" y="83.82"/>
+</segment>
+</net>
+<net name="QEB2" class="0">
+<segment>
+<pinref part="U1" gate="A" pin="RPB13/PWM2L/CTPLS/RB13"/>
+<wire x1="200.66" y1="68.58" x2="213.36" y2="68.58" width="0.1524" layer="91"/>
+<label x="215.9" y="68.58" size="1.778" layer="95"/>
+<junction x="200.66" y="68.58"/>
+<junction x="213.36" y="68.58"/>
+</segment>
+<segment>
+<wire x1="193.04" y1="86.36" x2="205.74" y2="86.36" width="0.1524" layer="91"/>
+<pinref part="J2" gate="G$1" pin="4"/>
+<label x="198.12" y="83.82" size="1.778" layer="95"/>
+<junction x="193.04" y="86.36"/>
+<junction x="205.74" y="86.36"/>
+</segment>
+</net>
+<net name="INDX2" class="0">
+<segment>
+<pinref part="U1" gate="A" pin="RPB12/PWM2H/RB12"/>
+<wire x1="200.66" y1="66.04" x2="213.36" y2="66.04" width="0.1524" layer="91"/>
+<label x="215.9" y="66.04" size="1.778" layer="95"/>
+<junction x="200.66" y="66.04"/>
+<junction x="213.36" y="66.04"/>
+</segment>
+<segment>
+<wire x1="193.04" y1="88.9" x2="205.74" y2="88.9" width="0.1524" layer="91"/>
+<pinref part="J2" gate="G$1" pin="6"/>
+<junction x="193.04" y="88.9"/>
+<junction x="205.74" y="88.9"/>
+<label x="198.12" y="86.36" size="1.778" layer="95"/>
+</segment>
+</net>

Commit message: up
Connections:
- new net PWM1H: J3.9, U1.RPB14/PWM1H/RB14
- new net PWM1L: J3.7, U1.RPB15/PWM1L/RB15
- new net PWM4H: J3.10, U1.TDO/PWM4H/RA10
- new net PWM4L: J3.8, U1.TCK/RPA7/PWM4L/RA7
- net VSS: now also J3.2
Changed lines of the file:
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@@
 <part name="J3" library="MLE-105-01-G-DV" deviceset="MLE-105-01-G-DV" device=""/>
 <part name="VSS13" library="supply1" library_urn="urn:adsk.eagle:library:371" deviceset="VSS" device=""/>
+<part name="VSS14" library="supply1" library_urn="urn:adsk.eagle:library:371" deviceset="VSS" device=""/>
 </parts>
 <sheets>
@@
 <instance part="VSS13" gate="G$1" x="170.18" y="-17.78" smashed="yes">
 <attribute name="VALUE" x="167.64" y="-22.86" size="1.778" layer="96" rot="R90"/>
+</instance>
+<instance part="VSS14" gate="G$1" x="193.04" y="-17.78" smashed="yes">
+<attribute name="VALUE" x="190.5" y="-22.86" size="1.778" layer="96" rot="R90"/>
 </instance>
 </instances>
@@
 <junction x="170.18" y="-15.24"/>
 </segment>
+<segment>
+<pinref part="J3" gate="G$1" pin="2"/>
+<pinref part="VSS14" gate="G$1" pin="VSS"/>
+<junction x="193.04" y="-15.24"/>
+</segment>
 </net>
 <net name="AVDD" class="0">
@@
 </segment>
 </net>
+<net name="PWM1L" class="0">
+<segment>
+<pinref part="U1" gate="A" pin="RPB15/PWM1L/RB15"/>
+<wire x1="-17.78" y1="66.04" x2="-30.48" y2="66.04" width="0.1524" layer="91"/>
+<label x="-43.18" y="66.04" size="1.778" layer="95"/>
+<junction x="-17.78" y="66.04"/>
+<junction x="-30.48" y="66.04"/>
+</segment>
+<segment>
+<wire x1="170.18" y1="-7.62" x2="157.48" y2="-7.62" width="0.1524" layer="91"/>
+<pinref part="J3" gate="G$1" pin="7"/>
+<label x="147.32" y="-7.62" size="1.778" layer="95"/>
+<junction x="170.18" y="-7.62"/>
+<junction x="157.48" y="-7.62"/>
+</segment>
+</net>
+<net name="PWM1H" class="0">
+<segment>
+<pinref part="U1" gate="A" pin="RPB14/PWM1H/RB14"/>
+<wire x1="-17.78" y1="68.58" x2="-30.48" y2="68.58" width="0.1524" layer="91"/>
+<label x="-43.18" y="68.58" size="1.778" layer="95"/>
+<junction x="-17.78" y="68.58"/>
+<junction x="-30.48" y="68.58"/>
+</segment>
+<segment>
+<wire x1="170.18" y1="-5.08" x2="157.48" y2="-5.08" width="0.1524" layer="91"/>
+<pinref part="J3" gate="G$1" pin="9"/>
+<label x="147.32" y="-5.08" size="1.778" layer="95"/>
+<junction x="170.18" y="-5.08"/>
+<junction x="157.48" y="-5.08"/>
+</segment>
+</net>
+<net name="PWM4L" class="0">
+<segment>
+<pinref part="U1" gate="A" pin="TCK/RPA7/PWM4L/RA7"/>
+<wire x1="-17.78" y1="71.12" x2="-30.48" y2="71.12" width="0.1524" layer="91"/>
+<label x="-43.18" y="71.12" size="1.778" layer="95"/>
+<junction x="-17.78" y="71.12"/>
+<junction x="-30.48" y="71.12"/>
+</segment>
+<segment>
+<wire x1="205.74" y1="-7.62" x2="193.04" y2="-7.62" width="0.1524" layer="91"/>
+<pinref part="J3" gate="G$1" pin="8"/>
+<label x="208.28" y="-7.62" size="1.778" layer="95"/>
+<junction x="193.04" y="-7.62"/>
+<junction x="205.74" y="-7.62"/>
+</segment>
+</net>
+<net name="PWM4H" class="0">
+<segment>
+<pinref part="U1" gate="A" pin="TDO/PWM4H/RA10"/>
+<wire x1="200.66" y1="71.12" x2="213.36" y2="71.12" width="0.1524" layer="91"/>
+<label x="215.9" y="71.12" size="1.778" layer="95"/>
+<junction x="200.66" y="71.12"/>
+<junction x="213.36" y="71.12"/>
+</segment>
+<segment>
+<wire x1="193.04" y1="-5.08" x2="205.74" y2="-5.08" width="0.1524" layer="91"/>
+<pinref part="J3" gate="G$1" pin="10"/>
+<label x="208.28" y="-5.08" size="1.778" layer="95"/>
+<junction x="193.04" y="-5.08"/>
+<junction x="205.74" y="-5.08"/>
+</segment>
+</net>

Commit message: up
Parts:
- added C10, C8, C9: 0.1uf, rcl:C-USC0805
- added C11: 10uf, rcl:C-USC0805
- added REFCLK2, TP1, TP2, TP3: PTR1PAD1-13, testpad:PTR1PAD1-13
- added U2: MAX6126B30, MAX6126B30:MAX6126B30
Connections:
- new net N$4: C8.1, U2.NR
- new net N$5: TP1.TP, U1.AN11/CVD11/C1IN2-/FLT4/RC11
- new net N$6: TP2.TP, U1.OA3IN+/AN8/CVD8/C3IN1+/C3IN3-/RPC2/FLT3/RC2
- new net N$7: TP3.TP, U1.PGD3/VREF-/OA2IN-/AN2/C2IN1-/RPB0/CTED2/RB0
- new net N$8: REFCLK2.TP, U1.OA5IN+/AN24/CVD24/C5IN1+/C5IN3-/RPA4/RA4
- new net PWM1EN: J3.5, U1.RD8
- new net PWM1ER: J3.3, U1.SOSCO/RPB8/T1CK/RB8
- new net PWM4EN: J3.6, U1.RPB11/PWM3L/RB11
- new net PWM4ER: J3.4, U1.TDI/DAC2/AN26/CVD26/RPA8/SDA2/RA8
- new net SCK1: J1.8, U1.OA5OUT/AN25/CVD25/C5IN4-/RPB7/SCK1/INT0/RB7
- net AVDD: now also C10.1, U2.IN
- net EXT_SW2: now also J2.8; no longer J1.8
- net QEA2: now also U1.RPB10/PWM3H/RB10; no longer U1.RPB11/PWM3L/RB11
- net U1TX: now also U1.OA3OUT/AN6/CVD6/C3IN4-/C4IN1+/C4IN4-/RPC0/RC0; no longer U1.OA3IN+/AN8/CVD8/C3IN1+/C3IN3-/RPC2/FLT3/RC2
- net VREF+: now also C11.1, C9.1, U2.OUTF, U2.OUTS
- net VSS: now also C10.2, C11.2, C8.2, C9.2, U2.GND, U2.GNDS
