File: wfipic32.sch (EAGLE design)
At the start: 30 parts, among them IC1 BMA490L, J1 MLE-105-01-G-DV, J2 MLE-105-01-G-DV, J3 MLE-105-01-G-DV, U1 PIC32MK0512MCJ048T-I/Y8XTQFP4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, U2 MAX6126B30

Commit message: up
Parts:
- R3: value 2k -> 10k
- R4: value 2k -> 56
Connections:
- removed net N$7: TP3.TP, U1.PGD3/VREF-/OA2IN-/AN2/C2IN1-/RPB0/CTED2/RB0
- new net BMA_INT2: IC1.INT2, TP3.TP, U1.PGD3/VREF-/OA2IN-/AN2/C2IN1-/RPB0/CTED2/RB0
Changed lines of the file:
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@@
 <part name="R1" library="rcl" library_urn="urn:adsk.eagle:library:334" deviceset="R-US_" device="M0805" package3d_urn="urn:adsk.eagle:package:23556/2" value="2k"/>
 <part name="R2" library="rcl" library_urn="urn:adsk.eagle:library:334" deviceset="R-US_" device="M0805" package3d_urn="urn:adsk.eagle:package:23556/2" value="2k"/>
-<part name="R3" library="rcl" library_urn="urn:adsk.eagle:library:334" deviceset="R-US_" device="M0805" package3d_urn="urn:adsk.eagle:package:23556/2" value="2k"/>
+<part name="R3" library="rcl" library_urn="urn:adsk.eagle:library:334" deviceset="R-US_" device="M0805" package3d_urn="urn:adsk.eagle:package:23556/2" value="10k"/>
 <part name="C6" library="rcl" library_urn="urn:adsk.eagle:library:334" deviceset="C-US" device="C0805" package3d_urn="urn:adsk.eagle:package:23617/2" value="0.1uf"/>
-<part name="R4" library="rcl" library_urn="urn:adsk.eagle:library:334" deviceset="R-US_" device="M0805" package3d_urn="urn:adsk.eagle:package:23556/2" value="2k"/>
+<part name="R4" library="rcl" library_urn="urn:adsk.eagle:library:334" deviceset="R-US_" device="M0805" package3d_urn="urn:adsk.eagle:package:23556/2" value="56"/>
 <part name="VDD2" library="supply1" library_urn="urn:adsk.eagle:library:371" deviceset="VDD" device=""/>
 <part name="VSS7" library="supply1" library_urn="urn:adsk.eagle:library:371" deviceset="VSS" device=""/>
@@
 <part name="TP2" library="testpad" library_urn="urn:adsk.eagle:library:385" deviceset="PTR1" device="PAD1-13" package3d_urn="urn:adsk.eagle:package:27946/1"/>
 <part name="REFCLK2" library="testpad" library_urn="urn:adsk.eagle:library:385" deviceset="PTR1" device="PAD1-13" package3d_urn="urn:adsk.eagle:package:27946/1"/>
+<part name="VSS20" library="supply1" library_urn="urn:adsk.eagle:library:371" deviceset="VSS" device=""/>
 </parts>
 <sheets>
@@
 <attribute name="VALUE" x="2.54" y="132.08" size="1.778" layer="96" rot="R90"/>
 </instance>
-<instance part="VSS1" gate="G$1" x="5.08" y="121.92" smashed="yes">
-<attribute name="VALUE" x="2.54" y="116.84" size="1.778" layer="96" rot="R90"/>
+<instance part="VSS1" gate="G$1" x="7.62" y="121.92" smashed="yes">
+<attribute name="VALUE" x="5.08" y="116.84" size="1.778" layer="96" rot="R90"/>
 </instance>
 <instance part="L1" gate="G$1" x="17.78" y="139.7" smashed="yes">
@@
 <attribute name="NAME" x="222.25" y="11.684" size="1.778" layer="95" rot="R180"/>
 <attribute name="TP_SIGNAL_NAME" x="218.44" y="13.97" size="1.778" layer="97" rot="R90"/>
+</instance>
+<instance part="VSS20" gate="G$1" x="91.44" y="137.16" smashed="yes" rot="R270">
+<attribute name="VALUE" x="86.36" y="139.7" size="1.778" layer="96"/>
 </instance>
 </instances>
@@
 <net name="VSS" class="0">
 <segment>
-<wire x1="5.08" y1="124.46" x2="10.16" y2="124.46" width="0.1524" layer="91"/>
+<wire x1="7.62" y1="124.46" x2="10.16" y2="124.46" width="0.1524" layer="91"/>
 <pinref part="C1" gate="G$1" pin="2"/>
 <wire x1="10.16" y1="124.46" x2="17.78" y2="124.46" width="0.1524" layer="91"/>
@@
 <label x="27.94" y="121.92" size="1.778" layer="95"/>
 <pinref part="VSS1" gate="G$1" pin="VSS"/>
-<junction x="5.08" y="124.46"/>
-</segment>
-<segment>
-<wire x1="93.98" y1="132.08" x2="93.98" y2="144.78" width="0.1524" layer="91"/>
+<junction x="7.62" y="124.46"/>
+</segment>
+<segment>
+<wire x1="93.98" y1="132.08" x2="93.98" y2="137.16" width="0.1524" layer="91"/>
 <pinref part="IC1" gate="G$1" pin="GND"/>
 <junction x="93.98" y="132.08"/>
 <junction x="93.98" y="144.78"/>
 <label x="88.9" y="142.24" size="1.778" layer="95"/>
-</segment>
-<segment>
+<wire x1="93.98" y1="137.16" x2="93.98" y2="144.78" width="0.1524" layer="91"/>
 <wire x1="96.52" y1="132.08" x2="96.52" y2="144.78" width="0.1524" layer="91"/>
 <pinref part="IC1" gate="G$1" pin="GNDIO"/>
 <junction x="96.52" y="132.08"/>
 <junction x="96.52" y="144.78"/>
-<label x="96.52" y="149.86" size="1.778" layer="95"/>
+<label x="91.44" y="147.32" size="1.778" layer="95"/>
+<wire x1="93.98" y1="132.08" x2="96.52" y2="132.08" width="0.1524" layer="91"/>
+<wire x1="93.98" y1="144.78" x2="96.52" y2="144.78" width="0.1524" layer="91"/>
+<pinref part="VSS20" gate="G$1" pin="VSS"/>
+<junction x="93.98" y="137.16"/>
 </segment>
 <segment>
@@
 </segment>
 </net>
-<net name="N$7" class="0">
+<net name="BMA_INT2" class="0">
 <segment>
 <pinref part="U1" gate="A" pin="PGD3/VREF-/OA2IN-/AN2/C2IN1-/RPB0/CTED2/RB0"/>
@@
 <junction x="-45.72" y="45.72"/>
 <junction x="-17.78" y="45.72"/>
-</segment>
-</net>
+<label x="-43.18" y="45.72" size="1.778" layer="95"/>
+</segment>
+<segment>
+<wire x1="109.22" y1="114.3" x2="137.16" y2="114.3" width="0.1524" layer="91"/>
+<pinref part="IC1" gate="G$1" pin="INT2"/>
+<junction x="109.22" y="114.3"/>
+<junction x="137.16" y="114.3"/>
+<label x="119.38" y="114.3" size="1.778" layer="95"/>
+</segment>
+</net>

Commit message: up
Changed lines of the file:
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@@
 <part name="VSS8" library="supply1" library_urn="urn:adsk.eagle:library:371" deviceset="VSS" device=""/>
 <part name="JP2" library="pinhead" library_urn="urn:adsk.eagle:library:325" deviceset="PINHD-1X6" device="" package3d_urn="urn:adsk.eagle:package:22472/2" value="ICSP"/>
-<part name="VDD3" library="supply1" library_urn="urn:adsk.eagle:library:371" deviceset="VDD" device=""/>
-<part name="VSS9" library="supply1" library_urn="urn:adsk.eagle:library:371" deviceset="VSS" device=""/>
 <part name="J1" library="MLE-105-01-G-DV" deviceset="MLE-105-01-G-DV" device=""/>
 <part name="J2" library="MLE-105-01-G-DV" deviceset="MLE-105-01-G-DV" device=""/>
@@
 <attribute name="VALUE" x="44.45" y="5.08" size="1.778" layer="96" rot="R180"/>
 </instance>
-<instance part="VDD3" gate="G$1" x="55.88" y="-10.16" smashed="yes" rot="R270">
-<attribute name="VALUE" x="53.34" y="-7.62" size="1.778" layer="96"/>
-</instance>
-<instance part="VSS9" gate="G$1" x="55.88" y="-7.62" smashed="yes" rot="R90">
-<attribute name="VALUE" x="60.96" y="-10.16" size="1.778" layer="96" rot="R180"/>
-</instance>
 <instance part="J1" gate="G$1" x="170.18" y="129.54" smashed="yes">
 <attribute name="NAME" x="189.23" y="137.16" size="1.778" layer="95" align="center-left"/>
@@
 </segment>
 <segment>
-<pinref part="JP2" gate="A" pin="2"/>
-<wire x1="40.64" y1="-10.16" x2="53.34" y2="-10.16" width="0.1524" layer="91"/>
-<pinref part="VDD3" gate="G$1" pin="VDD"/>
-<junction x="40.64" y="-10.16"/>
-<junction x="53.34" y="-10.16"/>
-</segment>
-<segment>
 <pinref part="J1" gate="G$1" pin="10"/>
 <pinref part="VDD4" gate="G$1" pin="VDD"/>
@@
 <wire x1="213.36" y1="93.98" x2="193.04" y2="93.98" width="0.1524" layer="91"/>
 <junction x="213.36" y="93.98"/>
+</segment>
+<segment>
+<wire x1="40.64" y1="-10.16" x2="53.34" y2="-10.16" width="0.1524" layer="91"/>
+<pinref part="JP2" gate="A" pin="2"/>
+<junction x="40.64" y="-10.16"/>
+<junction x="53.34" y="-10.16"/>
+<label x="58.42" y="-10.16" size="1.778" layer="95"/>
 </segment>
 </net>
@@
 <pinref part="VSS8" gate="G$1" pin="VSS"/>
 <junction x="-10.16" y="93.98"/>
-</segment>
-<segment>
-<pinref part="JP2" gate="A" pin="3"/>
-<wire x1="40.64" y1="-7.62" x2="53.34" y2="-7.62" width="0.1524" layer="91"/>
-<pinref part="VSS9" gate="G$1" pin="VSS"/>
-<junction x="40.64" y="-7.62"/>
-<junction x="53.34" y="-7.62"/>
+<junction x="-7.62" y="99.06"/>
 </segment>
 <segment>
@@
 <pinref part="VSS19" gate="G$1" pin="VSS"/>
 <junction x="129.54" y="-12.7"/>
+</segment>
+<segment>
+<wire x1="40.64" y1="-7.62" x2="53.34" y2="-7.62" width="0.1524" layer="91"/>
+<pinref part="JP2" gate="A" pin="3"/>
+<junction x="40.64" y="-7.62"/>
+<junction x="53.34" y="-7.62"/>
+<label x="58.42" y="-7.62" size="1.778" layer="95"/>
 </segment>
 </net>
@@
 <wire x1="-17.78" y1="101.6" x2="-7.62" y2="101.6" width="0.1524" layer="91"/>
 <pinref part="JP1" gate="G$1" pin="1"/>
+<junction x="-7.62" y="101.6"/>
 </segment>
 </net>
@@
 <wire x1="137.16" y1="-5.08" x2="137.16" y2="-17.78" width="0.1524" layer="91"/>
 <junction x="137.16" y="-17.78"/>
-<label x="142.24" y="-15.24" size="1.778" layer="95"/>
-</segment>
-</net>
+<label x="139.7" y="-20.32" size="1.778" layer="95"/>
+</segment>
+</net>

Commit message: up
Parts:
- added J4: MLE-105-01-G-DV, MLE-105-01-G-DV:MLE-105-01-G-DV
Connections:
- net BMA_INT2: now also J4.6
- net EXT_INT2: now also J4.5
- net IMU_CS: now also J4.9
- net SCK2: now also J4.10
- net SDI2: now also J4.1
- net SDO2: now also J4.2
- net VDD: now also J4.3, J4.7
- net VSS: now also J4.8
Changed lines of the file:
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@@
 <part name="REFCLK2" library="testpad" library_urn="urn:adsk.eagle:library:385" deviceset="PTR1" device="PAD1-13" package3d_urn="urn:adsk.eagle:package:27946/1"/>
 <part name="VSS20" library="supply1" library_urn="urn:adsk.eagle:library:371" deviceset="VSS" device=""/>
+<part name="J4" library="MLE-105-01-G-DV" deviceset="MLE-105-01-G-DV" device=""/>
+<part name="VSS9" library="supply1" library_urn="urn:adsk.eagle:library:371" deviceset="VSS" device=""/>
 </parts>
 <sheets>
@@
 <instance part="VSS20" gate="G$1" x="91.44" y="137.16" smashed="yes" rot="R270">
 <attribute name="VALUE" x="86.36" y="139.7" size="1.778" layer="96"/>
+</instance>
+<instance part="J4" gate="G$1" x="132.08" y="147.32" smashed="yes">
+<attribute name="NAME" x="151.13" y="154.94" size="1.778" layer="95" align="center-left"/>
+<attribute name="VALUE" x="151.13" y="152.4" size="1.778" layer="96" align="center-left"/>
+</instance>
+<instance part="VSS9" gate="G$1" x="93.98" y="139.7" smashed="yes" rot="R270">
+<attribute name="VALUE" x="88.9" y="142.24" size="1.778" layer="96"/>
 </instance>
 </instances>
@@
 <label x="58.42" y="-10.16" size="1.778" layer="95"/>
 </segment>
+<segment>
+<wire x1="132.08" y1="139.7" x2="121.92" y2="139.7" width="0.1524" layer="91"/>
+<pinref part="J4" gate="G$1" pin="3"/>
+<label x="124.46" y="139.7" size="1.778" layer="95"/>
+<junction x="132.08" y="139.7"/>
+</segment>
+<segment>
+<wire x1="132.08" y1="144.78" x2="119.38" y2="144.78" width="0.1524" layer="91"/>
+<pinref part="J4" gate="G$1" pin="7"/>
+<label x="121.92" y="144.78" size="1.778" layer="95"/>
+<junction x="132.08" y="144.78"/>
+</segment>
 </net>
 <net name="VSS" class="0">
@@
 </segment>
 <segment>
+<pinref part="VSS20" gate="G$1" pin="VSS"/>
 <wire x1="93.98" y1="132.08" x2="93.98" y2="137.16" width="0.1524" layer="91"/>
 <pinref part="IC1" gate="G$1" pin="GND"/>
-<junction x="93.98" y="132.08"/>
-<junction x="93.98" y="144.78"/>
 <label x="88.9" y="142.24" size="1.778" layer="95"/>
-<wire x1="93.98" y1="137.16" x2="93.98" y2="144.78" width="0.1524" layer="91"/>
-<wire x1="96.52" y1="132.08" x2="96.52" y2="144.78" width="0.1524" layer="91"/>
-<pinref part="IC1" gate="G$1" pin="GNDIO"/>
-<junction x="96.52" y="132.08"/>
-<junction x="96.52" y="144.78"/>
 <label x="91.44" y="147.32" size="1.778" layer="95"/>
-<wire x1="93.98" y1="132.08" x2="96.52" y2="132.08" width="0.1524" layer="91"/>
-<wire x1="93.98" y1="144.78" x2="96.52" y2="144.78" width="0.1524" layer="91"/>
-<pinref part="VSS20" gate="G$1" pin="VSS"/>
 <junction x="93.98" y="137.16"/>
 </segment>
@@
 <junction x="53.34" y="-7.62"/>
 <label x="58.42" y="-7.62" size="1.778" layer="95"/>
+</segment>
+<segment>
+<wire x1="167.64" y1="144.78" x2="154.94" y2="144.78" width="0.1524" layer="91"/>
+<pinref part="J4" gate="G$1" pin="8"/>
+<label x="167.64" y="144.78" size="1.778" layer="95"/>
+<junction x="154.94" y="144.78"/>
+</segment>
+<segment>
+<wire x1="96.52" y1="132.08" x2="96.52" y2="139.7" width="0.1524" layer="91"/>
+<pinref part="IC1" gate="G$1" pin="GNDIO"/>
+<pinref part="VSS9" gate="G$1" pin="VSS"/>
+<junction x="96.52" y="139.7"/>
 </segment>
 </net>
@@
 <junction x="78.74" y="132.08"/>
 </segment>
+<segment>
+<wire x1="119.38" y1="147.32" x2="132.08" y2="147.32" width="0.1524" layer="91"/>
+<pinref part="J4" gate="G$1" pin="9"/>
+<label x="121.92" y="147.32" size="1.778" layer="95"/>
+<junction x="132.08" y="147.32"/>
+</segment>
 </net>
 <net name="N$3" class="0">
@@
 <junction x="68.58" y="111.76"/>
 </segment>
+<segment>
+<wire x1="154.94" y1="147.32" x2="167.64" y2="147.32" width="0.1524" layer="91"/>
+<pinref part="J4" gate="G$1" pin="10"/>
+<label x="165.1" y="147.32" size="1.778" layer="95"/>
+<junction x="154.94" y="147.32"/>
+</segment>
 </net>
 <net name="SDO2" class="0">
@@
 <junction x="93.98" y="81.28"/>
 </segment>
+<segment>
+<wire x1="167.64" y1="137.16" x2="154.94" y2="137.16" width="0.1524" layer="91"/>
+<pinref part="J4" gate="G$1" pin="2"/>
+<label x="165.1" y="137.16" size="1.778" layer="95"/>
+<junction x="154.94" y="137.16"/>
+</segment>
 </net>
 <net name="SDI2" class="0">
@@
 <junction x="91.44" y="93.98"/>
 <junction x="78.74" y="93.98"/>
+</segment>
+<segment>
+<wire x1="119.38" y1="137.16" x2="132.08" y2="137.16" width="0.1524" layer="91"/>
+<pinref part="J4" gate="G$1" pin="1"/>
+<label x="121.92" y="137.16" size="1.778" layer="95"/>
+<junction x="132.08" y="137.16"/>
 </segment>
 </net>
@@
 <junction x="121.92" y="111.76"/>
 <label x="116.84" y="109.22" size="1.778" layer="95"/>
+</segment>
+<segment>
+<wire x1="119.38" y1="142.24" x2="132.08" y2="142.24" width="0.1524" layer="91"/>
+<pinref part="J4" gate="G$1" pin="5"/>
+<label x="121.92" y="142.24" size="1.778" layer="95"/>
+<junction x="132.08" y="142.24"/>
 </segment>
 </net>
@@
 <junction x="170.18" y="-5.08"/>
 <junction x="157.48" y="-5.08"/>
+<junction x="170.18" y="-5.08"/>
+<junction x="170.18" y="-5.08"/>
 </segment>
 </net>
@@
 <label x="119.38" y="114.3" size="1.778" layer="95"/>
 </segment>
-</net>
+<segment>
+<wire x1="154.94" y1="142.24" x2="182.88" y2="142.24" width="0.1524" layer="91"/>
+<pinref part="J4" gate="G$1" pin="6"/>
+<label x="180.34" y="142.24" size="1.778" layer="95"/>
+<junction x="154.94" y="142.24"/>
+</segment>
+</net>
