File: wfipic32host.brd (EAGLE design)
At the start: 35.5 x 27.6 mm, 40 parts, among them IC1 BMA490L, IC2 TCAN330GD, J1 MLE-105-01-G-DV, J2 MLE-105-01-G-DV, J3 MLE-105-01-G-DV, J4 MLE-105-01-G-DV, U1 PIC32MK0512MCJ048T-I/Y8XTQFP4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, U2 MAX6126B30

Commit message: up
Parts:
- added C14, C16: 10uf, rcl:C0805
- added C15, C17: 0.1uf, rcl:C0805
- added SV1: ETH1, con-lstb:MA07-1
- added SV4, SV5: ETHG, con-lstb:MA03-1
- JP3: value RESET_JMP -> SIL
- JP4: value RESET_JMP -> STB
- moved JP5 60.5 mm to (-58.4, 29.2), turned to 90 degrees
- moved R5 55.7 mm to (-49.5, 27.9), turned to 90 degrees
- moved S1 33.5 mm to (-41.9, 26.7)
- moved JP4 25.4 mm to (-21.6, 22.9)
- moved JP3 22.5 mm to (-21.6, 26.7)
- moved C5 15.5 mm to (21.6, 31.8)
- moved J1 10.9 mm to (24.1, 24.1)
- moved IC2 8.52 mm to (-7.62, 25.4)
- moved C2 6.35 mm to (3.81, 24.1)
- moved J3 6.35 mm to (24.1, 54.6)
- moved LED1 5.24 mm to (2.54, 55.9)
- moved LED2 5.24 mm to (2.54, 58.4)
- moved C1 5.08 mm to (3.81, 27.9)
- moved J4 5.08 mm to (20.3, 54.6)
- moved JP1 5.08 mm to (12.7, 57.1)
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Connections:
- net U1RX: now also SV1.3
- net U1TX: now also SV1.2
- net VDD: now also C14.1, C15.1, C16.1, C17.1, SV1.6
- net VSS: now also C14.2, C15.2, C16.2, C17.2, SV1.5, SV4.1, SV4.2, SV4.3, SV5.1, SV5.2, SV5.3
Routing:
- net VDD: track 140.7 -> 285.7 mm, vias 6 -> 5
- net PGD_C1TX: track 33.0 -> 137.8 mm, vias 1 -> 0
- net PGC_C1RX: track 34.3 -> 118.1 mm, vias 1 -> 2
- net CANL: track 0.00 -> 59.3 mm
- net CANH: track 0.00 -> 57.3 mm, vias 0 -> 1
- net VSS: track 131.3 -> 186.0 mm, vias 5 -> 7
- net U1RX: track 23.6 -> 71.4 mm, vias 2 -> 0
- net AVDD: track 75.3 -> 32.9 mm
- net BMA_INT2: track 107.9 -> 65.8 mm, vias 1 -> 2
- net EXT_SW2: track 17.4 -> 49.2 mm, vias 2 -> 0
- net N$10: track 0.00 -> 30.0 mm
- net N$11: track 0.00 -> 29.9 mm
- net PWM4ER: track 27.1 -> 53.2 mm
- net U1TX: track 18.4 -> 41.3 mm
- net RED_LED: track 19.1 -> 41.4 mm
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Other:
- board size 35.5 x 27.6 mm -> 95.2 x 42.9 mm
- board text added: "CAN-FD ON"
- board text added: "PIC32MK-CANFD HOST V1.5"
- board text removed: "BMA490L-PIC32MK V1.3"

Commit message: up
Parts:
- removed REFCLK2: PTR1PAD1-13, testpad:P1-13
- added 3.3VDC: 3.3 Vreg, linear:TO220V
- added C18, C19, C20: 0.1uf, rcl:C0805
- added C21, C22: 10uf, rcl:C0805
- added GLED: PTR1PAD1-13, testpad:P1-13
- added JP6: DC5+, pinhead:1X02
- added OS1: OSC-OE-CFPS-32, IQD-Frequency-Products:7.2X5.2-4-PAD
- added R6: 0 ohm fuse, rcl:M1206
- moved TP3 32.9 mm to (-1.27, 52.1)
- moved C13 2.54 mm to (26.7, 34.3)
- moved J2 2.54 mm to (24.1, 45.7)
- moved JP2 2.54 mm to (33.0, 43.2)
- moved U1 1.80 mm to (11.4, 39.4)
- moved R4 1.27 mm to (0.00, 41.9), turned to 0 degrees
- moved C14 1.27 mm to (-16.5, 24.1)
- moved C15 1.27 mm to (-14.0, 24.1)
- moved C7 1.27 mm to (26.7, 31.8)
- moved IC2 1.27 mm to (-7.62, 24.1)
- moved J1 1.27 mm to (25.4, 24.1)
- turned JP1 to 0 degrees
Connections:
- removed net N$8: REFCLK2.TP, U1.25
- new net DC_IN: JP6.2, R6.2
- new net DC_INPUT: 3.3VDC.1, C20.1, C21.1, R6.1
- new net OSC_MCU: OS1.3, U1.27
- net GREEN_LED: now also GLED.TP, U1.25; no longer U1.27
- net VDD: now also 3.3VDC.3, C18.1, C19.1, C22.1, OS1.1, OS1.4
- net VSS: now also 3.3VDC.2, C18.2, C19.2, C20.2, C21.2, C22.2, JP6.1, OS1.2
Routing:
- net PGD_C1TX: track 137.8 -> 89.4 mm, vias 0 -> 2
- net DC_INPUT: track 0.00 -> 34.5 mm
- net VSS: track 186.0 -> 220.3 mm
- net EXT_SW2: track 49.2 -> 19.7 mm
- net OSC_MCU: track 0.00 -> 29.3 mm, vias 0 -> 2
- net AN0: track 21.0 -> 44.4 mm
- net PGC_C1RX: track 118.1 -> 95.7 mm
- net U1RX: track 71.4 -> 49.5 mm, vias 0 -> 2
- net VDD: track 285.7 -> 307.0 mm, vias 5 -> 2
- net PWM4ER: track 53.2 -> 35.2 mm
- net PWM1H: track 21.3 -> 38.5 mm
- net SCK2: track 39.7 -> 23.9 mm, vias 2 -> 3
- net BMA_INT2: track 65.8 -> 50.7 mm, vias 2 -> 3
- net RED_LED: track 41.4 -> 26.7 mm
- net INDX2: track 37.1 -> 23.5 mm
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
Commit message: up
Connections:
- net VDD: now also IC2.3; no longer IC2.2
- net VSS: now also IC2.2; no longer IC2.3
Routing:
- net VDD: track 307.0 -> 310.1 mm
- net VSS: track 220.3 -> 221.7 mm
Other:
- board text added: "PIC32MK-CANFD HOST V1.6"
- board text removed: "PIC32MK-CANFD HOST V1.5"
Changed lines of the file:
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@@
 <wire x1="36.81" y1="60.63" x2="-58.42" y2="60.63" width="0" layer="20"/>
 <wire x1="-58.42" y1="60.63" x2="-58.42" y2="17.78" width="0" layer="20"/>
-<text x="15.24" y="20.32" size="1.016" layer="1" font="vector" ratio="17" distance="77" rot="R180">PIC32MK-CANFD HOST V1.5</text>
+<text x="11.43" y="20.32" size="1.016" layer="1" font="vector" ratio="17" distance="77" rot="R180">PIC32MK-CANFD HOST V1.6</text>
 <hole x="-55.88" y="20.32" drill="2.54"/>
 <hole x="-55.88" y="58.42" drill="2.54"/>
@@
 </element>
 <element name="3.3VDC" library="linear" library_urn="urn:adsk.eagle:library:262" package="TO220V" package3d_urn="urn:adsk.eagle:package:16417/2" value="3.3 Vreg" x="13.97" y="25.4" smashed="yes">
-<attribute name="NAME" x="8.89" y="19.3548" size="1.27" layer="25" ratio="10"/>
+<attribute name="NAME" x="12.7" y="19.3548" size="1.27" layer="25" ratio="10"/>
 <attribute name="POPULARITY" value="57" x="13.97" y="25.4" size="1.778" layer="27" display="off"/>
 <attribute name="VALUE" x="8.89" y="17.78" size="1.27" layer="27" ratio="10"/>
@@
 <contactref element="J4" pad="7"/>
 <contactref element="AC1" pad="9"/>
-<contactref element="IC2" pad="2"/>
 <contactref element="JP3" pad="1"/>
 <contactref element="JP4" pad="1"/>
@@
 <wire x1="-16.4592" y1="25.0698" x2="-16.51" y2="25.08" width="0.1524" layer="1"/>
 <wire x1="-14.0208" y1="25.0698" x2="-13.97" y2="25.08" width="0.1524" layer="1"/>
-<wire x1="-13.6398" y1="24.765" x2="-10.331" y2="24.765" width="0.1524" layer="1"/>
 <wire x1="-13.9446" y1="25.0698" x2="-13.6398" y2="24.765" width="0.1524" layer="1"/>
 <wire x1="-13.9446" y1="25.0698" x2="-13.97" y2="25.08" width="0.1524" layer="1"/>
@@
 <wire x1="-3.1623" y1="26.3271" x2="-3.429" y2="26.5938" width="0.1524" layer="1"/>
 <wire x1="-2.286" y1="25.4508" x2="-2.22" y2="25.4" width="0.1524" layer="1"/>
-<wire x1="-6.3246" y1="24.765" x2="-10.331" y2="24.765" width="0.1524" layer="1"/>
-<wire x1="-5.6388" y1="25.4508" x2="-6.3246" y2="24.765" width="0.1524" layer="1"/>
-<wire x1="-4.0386" y1="25.4508" x2="-5.6388" y2="25.4508" width="0.1524" layer="1"/>
-<wire x1="-3.1623" y1="26.3271" x2="-4.0386" y2="25.4508" width="0.1524" layer="1"/>
 <wire x1="-22.86" y1="26.67" x2="-22.86" y2="22.86" width="0.1524" layer="16"/>
 <wire x1="-29.1846" y1="32.9946" x2="-54.5592" y2="32.9946" width="0.1524" layer="1"/>
@@
 <via x="20.1168" y="47.4726" extent="1-16" drill="0.35"/>
 <via x="23.5458" y="31.7754" extent="1-16" drill="0.35"/>
+<contactref element="IC2" pad="3"/>
+<wire x1="-4.0386" y1="25.4508" x2="-11.1252" y2="25.4508" width="0.1524" layer="1"/>
+<wire x1="-3.1623" y1="26.3271" x2="-4.0386" y2="25.4508" width="0.1524" layer="1"/>
+<wire x1="-13.6398" y1="24.8412" x2="-13.97" y2="25.08" width="0.1524" layer="1"/>
+<wire x1="-10.5918" y1="23.5458" x2="-10.3632" y2="23.5458" width="0.1524" layer="1"/>
+<wire x1="-10.3632" y1="23.5458" x2="-10.331" y2="23.495" width="0.1524" layer="1"/>
+<wire x1="-11.3538" y1="24.3078" x2="-10.5918" y2="23.5458" width="0.1524" layer="1"/>
+<wire x1="-11.3538" y1="25.2222" x2="-11.3538" y2="24.8412" width="0.1524" layer="1"/>
+<wire x1="-11.3538" y1="24.8412" x2="-11.3538" y2="24.3078" width="0.1524" layer="1"/>
+<wire x1="-11.1252" y1="25.4508" x2="-11.3538" y2="25.2222" width="0.1524" layer="1"/>
+<wire x1="-10.5918" y1="23.5458" x2="-10.331" y2="23.495" width="0.1524" layer="1"/>
+<wire x1="-13.5636" y1="24.8412" x2="-11.3538" y2="24.8412" width="0.1524" layer="1"/>
+<wire x1="-13.5636" y1="24.8412" x2="-13.97" y2="25.08" width="0.1524" layer="1"/>
 </signal>
 <signal name="VSS">
@@
 <contactref element="C13" pad="2"/>
 <contactref element="AC1" pad="3"/>
-<contactref element="IC2" pad="3"/>
 <contactref element="JP5" pad="2"/>
 <contactref element="SV1" pad="5"/>
@@
 <wire x1="-16.4592" y1="23.1648" x2="-16.51" y2="23.18" width="0.1524" layer="1"/>
 <wire x1="-14.0208" y1="23.1648" x2="-13.97" y2="23.18" width="0.1524" layer="1"/>
-<wire x1="-10.1346" y1="23.4696" x2="-10.287" y2="23.4696" width="0.1524" layer="1"/>
-<wire x1="-9.2964" y1="22.6314" x2="-10.1346" y2="23.4696" width="0.1524" layer="1"/>
-<wire x1="-9.2964" y1="21.7932" x2="-9.2964" y2="22.6314" width="0.1524" layer="1"/>
-<wire x1="-9.4488" y1="21.6408" x2="-9.2964" y2="21.7932" width="0.1524" layer="1"/>
-<wire x1="-12.4206" y1="21.6408" x2="-9.4488" y2="21.6408" width="0.1524" layer="1"/>
-<wire x1="-13.9446" y1="23.1648" x2="-12.8778" y2="22.098" width="0.1524" layer="1"/>
-<wire x1="-12.8778" y1="22.098" x2="-12.4206" y2="21.6408" width="0.1524" layer="1"/>
-<wire x1="-10.287" y1="23.4696" x2="-10.331" y2="23.495" width="0.1524" layer="1"/>
 <wire x1="-13.9446" y1="23.1648" x2="-13.97" y2="23.18" width="0.1524" layer="1"/>
 <wire x1="21.4884" y1="45.8724" x2="20.574" y2="45.8724" width="0.1524" layer="16"/>
@@
 <via x="10.2108" y="33.7566" extent="1-16" drill="0.35"/>
 <via x="2.8956" y="21.6408" extent="1-16" drill="0.35"/>
-<via x="-12.8778" y="22.098" extent="1-16" drill="0.35"/>
+<contactref element="IC2" pad="2"/>
+<wire x1="-10.1346" y1="24.765" x2="-10.331" y2="24.765" width="0.1524" layer="1"/>
+<wire x1="-9.2964" y1="23.9268" x2="-10.1346" y2="24.765" width="0.1524" layer="1"/>
+<wire x1="-9.2964" y1="21.7932" x2="-9.2964" y2="23.9268" width="0.1524" layer="1"/>
+<wire x1="-9.4488" y1="21.6408" x2="-9.2964" y2="21.7932" width="0.1524" layer="1"/>
+<wire x1="-12.3444" y1="21.6408" x2="-9.4488" y2="21.6408" width="0.1524" layer="1"/>
+<wire x1="-13.8684" y1="23.1648" x2="-12.8397" y2="22.1361" width="0.1524" layer="1"/>
+<wire x1="-12.8397" y1="22.1361" x2="-12.3444" y2="21.6408" width="0.1524" layer="1"/>
+<wire x1="-13.8684" y1="23.1648" x2="-13.97" y2="23.18" width="0.1524" layer="1"/>
+<wire x1="-12.8016" y1="22.1742" x2="-12.8397" y2="22.1361" width="0.1524" layer="1"/>
+<via x="-12.8016" y="22.1742" extent="1-16" drill="0.35"/>
 </signal>
 <signal name="AVDD">

Commit message: up
Parts:
- added SV2: GLCD, con-lstb:MA10-1
- moved JP3 5.08 mm to (-21.6, 31.8)
- moved JP4 3.81 mm to (-21.6, 26.7)
- moved S1 2.84 mm to (-40.6, 29.2)
- moved R5 1.27 mm to (-49.5, 29.2)
Connections:
- net EXT_SW1: now also SV2.5
- net SCK1: now also SV2.3
- net SDI1: now also SV2.1
- net SDI1_MODE: now also SV2.6
- net SDO1: now also SV2.2
- net SS1_OUT: now also SV2.4
- net VDD: now also SV2.7
- net VSS: now also SV2.8
Routing:
- net SCK1: track 21.9 -> 103.5 mm
- net SDI1: track 17.7 -> 97.3 mm, vias 0 -> 3
- net SDI1_MODE: track 24.6 -> 99.0 mm
- net SDO1: track 27.7 -> 99.6 mm, vias 2 -> 3
- net SS1_OUT: track 22.7 -> 93.8 mm
- net EXT_SW1: track 24.4 -> 89.5 mm, vias 2 -> 3
- net VREF+: track 57.6 -> 82.5 mm
- net GREEN_LED: track 37.7 -> 58.1 mm, vias 2 -> 1
- net PWM1L: track 24.3 -> 41.4 mm, vias 2 -> 0
- net MCLR_SIG: track 49.9 -> 65.1 mm, vias 1 -> 0
- net VSS: track 221.7 -> 235.8 mm, vias 7 -> 4
- net IMU_CS: track 30.9 -> 44.8 mm, vias 4 -> 3
- net AN0: track 44.4 -> 30.8 mm
- net SCK2: track 23.9 -> 36.2 mm, vias 3 -> 2
- net RED_LED: track 26.7 -> 37.5 mm, vias 2 -> 3
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
Commit message: up
Parts:
- added 3.3VTP, GND_TP, OSCI, VREF_TP: PTR1PAD1-13, testpad:P1-13
- added C23: 10uf, rcl:C0805
- JP6: value DC5+ -> DC12+
Connections:
- net AVDD: now also C23.1
- net OSC_MCU: now also OSCI.TP
- net VDD: now also 3.3VTP.TP
- net VREF+: now also VREF_TP.TP
- net VSS: now also C23.2, GND_TP.TP
Routing:
- net VREF+: track 82.5 -> 97.3 mm
- net VDD: track 319.3 -> 332.1 mm
- net OSC_MCU: track 31.6 -> 39.7 mm
- net VSS: track 235.8 -> 243.8 mm
- net AVDD: track 35.3 -> 41.8 mm
Changed lines of the file:
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@@
 <attribute name="MFR_NAME" value="Microchip" x="67.31" y="19.05" size="1.778" layer="27" display="off"/>
 <attribute name="NAME" x="17.0488" y="33.655" size="1.27" layer="27" ratio="6"/>
-<attribute name="VALUE" x="3.3512" y="47.625" size="1.27" layer="21" ratio="6"/>
+<attribute name="VALUE" x="-47.4488" y="57.785" size="1.27" layer="21" ratio="6"/>
 </element>
 <element name="IC1" library="SamacSys_Parts" package="BMA490L" value="BMA490L" x="12.7" y="48.26" smashed="yes" rot="MR0">
@@
 <attribute name="VALUE" x="20.32" y="17.78" size="1.27" layer="28" rot="MR0"/>
 </element>
-<element name="JP6" library="pinhead" library_urn="urn:adsk.eagle:library:325" package="1X02" package3d_urn="urn:adsk.eagle:package:22435/2" value="DC5+" x="33.02" y="25.4" smashed="yes" rot="R90">
+<element name="JP6" library="pinhead" library_urn="urn:adsk.eagle:library:325" package="1X02" package3d_urn="urn:adsk.eagle:package:22435/2" value="DC12+" x="33.02" y="25.4" smashed="yes" rot="R90">
 <attribute name="NAME" x="31.1912" y="22.7838" size="1.27" layer="25" ratio="10" rot="R90"/>
 <attribute name="POPULARITY" value="98" x="33.02" y="25.4" size="1.778" layer="27" rot="R90" display="off"/>
@@
 <attribute name="POPULARITY" value="4" x="-35.56" y="21.59" size="1.778" layer="27" display="off"/>
 <attribute name="VALUE" x="-34.29" y="18.669" size="1.27" layer="27" ratio="10"/>
+</element>
+<element name="OSCI" library="testpad" library_urn="urn:adsk.eagle:library:385" package="P1-13" package3d_urn="urn:adsk.eagle:package:27946/1" value="PTR1PAD1-13" x="-12.7" y="38.1" smashed="yes" rot="MR0">
+<attribute name="NAME" x="-11.684" y="39.37" size="1.27" layer="26" ratio="10" rot="MR0"/>
+<attribute name="POPULARITY" value="2" x="-12.7" y="38.1" size="1.778" layer="28" rot="MR0" display="off"/>
+<attribute name="TP_SIGNAL_NAME" value="" x="-12.7" y="38.1" size="1.778" layer="28" rot="MR0" display="off"/>
+<attribute name="VALUE" x="-12.7" y="38.1" size="0.0254" layer="28" rot="MR0"/>
+</element>
+<element name="3.3VTP" library="testpad" library_urn="urn:adsk.eagle:library:385" package="P1-13" package3d_urn="urn:adsk.eagle:package:27946/1" value="PTR1PAD1-13" x="-43.18" y="45.72" smashed="yes" rot="MR0">
+<attribute name="NAME" x="-42.164" y="46.99" size="1.27" layer="26" ratio="10" rot="MR0"/>
+<attribute name="POPULARITY" value="2" x="-43.18" y="45.72" size="1.778" layer="28" rot="MR0" display="off"/>
+<attribute name="TP_SIGNAL_NAME" value="" x="-43.18" y="45.72" size="1.778" layer="28" rot="MR0" display="off"/>
+<attribute name="VALUE" x="-43.18" y="45.72" size="0.0254" layer="28" rot="MR0"/>
+</element>
+<element name="GND_TP" library="testpad" library_urn="urn:adsk.eagle:library:385" package="P1-13" package3d_urn="urn:adsk.eagle:package:27946/1" value="PTR1PAD1-13" x="-33.02" y="45.72" smashed="yes" rot="MR0">
+<attribute name="NAME" x="-32.004" y="46.99" size="1.27" layer="26" ratio="10" rot="MR0"/>
+<attribute name="POPULARITY" value="2" x="-33.02" y="45.72" size="1.778" layer="28" rot="MR0" display="off"/>
+<attribute name="TP_SIGNAL_NAME" value="" x="-33.02" y="45.72" size="1.778" layer="28" rot="MR0" display="off"/>
+<attribute name="VALUE" x="-33.02" y="45.72" size="0.0254" layer="28" rot="MR0"/>
+</element>
+<element name="VREF_TP" library="testpad" library_urn="urn:adsk.eagle:library:385" package="P1-13" package3d_urn="urn:adsk.eagle:package:27946/1" value="PTR1PAD1-13" x="-22.86" y="45.72" smashed="yes" rot="MR0">
+<attribute name="NAME" x="-21.844" y="46.99" size="1.27" layer="26" ratio="10" rot="MR0"/>
+<attribute name="POPULARITY" value="2" x="-22.86" y="45.72" size="1.778" layer="28" rot="MR0" display="off"/>
+<attribute name="TP_SIGNAL_NAME" value="" x="-22.86" y="45.72" size="1.778" layer="28" rot="MR0" display="off"/>
+<attribute name="VALUE" x="-22.86" y="45.72" size="0.0254" layer="28" rot="MR0"/>
+</element>
+<element name="C23" library="rcl" library_urn="urn:adsk.eagle:library:334" package="C0805" package3d_urn="urn:adsk.eagle:package:23617/2" value="10uf" x="-1.27" y="30.48" smashed="yes" rot="R180">
+<attribute name="NAME" x="0" y="29.21" size="1.27" layer="25" rot="R180"/>
+<attribute name="POPULARITY" value="63" x="-1.27" y="30.48" size="1.778" layer="27" rot="R180" display="off"/>
+<attribute name="SPICEPREFIX" value="C" x="-1.27" y="30.48" size="1.778" layer="27" rot="R180" display="off"/>
+<attribute name="VALUE" x="0" y="33.02" size="1.27" layer="27" rot="R180"/>
 </element>
 </elements>
@@
 <via x="4.7244" y="21.6408" extent="1-16" drill="0.35"/>
 <wire x1="-11.43" y1="33.528" x2="-11.43" y2="33.85" width="0.1524" layer="1"/>
+<contactref element="3.3VTP" pad="TP"/>
+<wire x1="-43.1292" y1="32.9946" x2="-43.1292" y2="45.72" width="0.1524" layer="15"/>
+<wire x1="-43.1292" y1="45.72" x2="-43.18" y2="45.72" width="0.1524" layer="15"/>
 </signal>
 <signal name="VSS">
@@
 <via x="8.4582" y="40.1574" extent="1-16" drill="0.35"/>
 <via x="27.5844" y="37.1856" extent="1-16" drill="0.35"/>
+<contactref element="GND_TP" pad="TP"/>
+<contactref element="C23" pad="2"/>
+<wire x1="-2.0574" y1="30.48" x2="-2.22" y2="30.48" width="0.1524" layer="1"/>
+<wire x1="-0.5334" y1="28.956" x2="-2.0574" y2="30.48" width="0.1524" layer="1"/>
+<wire x1="3.5814" y1="28.956" x2="-0.5334" y2="28.956" width="0.1524" layer="1"/>
+<wire x1="4.6482" y1="27.8892" x2="3.5814" y2="28.956" width="0.1524" layer="1"/>
+<wire x1="4.6482" y1="27.8892" x2="4.76" y2="27.94" width="0.1524" layer="1"/>
 </signal>
 <signal name="AVDD">
@@
 <via x="9.2202" y="36.4236" extent="1-16" drill="0.35"/>
 <via x="11.2776" y="27.9654" extent="1-16" drill="0.35"/>
+<contactref element="C23" pad="1"/>
+<wire x1="5.4102" y1="30.48" x2="-0.32" y2="30.48" width="0.1524" layer="1"/>
+<wire x1="5.9436" y1="29.9466" x2="5.4102" y2="30.48" width="0.1524" layer="1"/>
 </signal>
 <signal name="N$1">
@@
 <via x="18.4404" y="39.4716" extent="1-16" drill="0.35"/>
 <via x="-1.4478" y="36.0426" extent="1-16" drill="0.35"/>
+<contactref element="OSCI" pad="TP"/>
+<wire x1="-10.5918" y1="38.1" x2="-12.7" y2="38.1" width="0.1524" layer="1"/>
+<wire x1="-6.4008" y1="33.909" x2="-10.5918" y2="38.1" width="0.1524" layer="1"/>
+<wire x1="-6.4008" y1="33.909" x2="-6.35" y2="33.85" width="0.1524" layer="1"/>
 </signal>
 <signal name="RED_LED">
@@
 <wire x1="-7.5438" y1="53.1114" x2="-5.1816" y2="53.1114" width="0.1524" layer="16"/>
 <wire x1="-8.1534" y1="52.5018" x2="-7.5438" y2="53.1114" width="0.1524" layer="16"/>
-<wire x1="-8.1534" y1="38.9382" x2="-8.1534" y2="52.5018" width="0.1524" layer="16"/>
+<wire x1="-8.1534" y1="38.9382" x2="-8.1534" y2="45.72" width="0.1524" layer="16"/>
+<wire x1="-8.1534" y1="45.72" x2="-8.1534" y2="52.5018" width="0.1524" layer="16"/>
 <wire x1="0" y1="30.7848" x2="-8.1534" y2="38.9382" width="0.1524" layer="16"/>
 <wire x1="2.8194" y1="30.7848" x2="0" y2="30.7848" width="0.1524" layer="16"/>
@@
 <via x="4.572" y="34.5186" extent="1-16" drill="0.35"/>
 <via x="11.2776" y="37.0332" extent="1-16" drill="0.35"/>
+<contactref element="VREF_TP" pad="TP"/>
+<wire x1="-8.1534" y1="45.72" x2="-22.86" y2="45.72" width="0.1524" layer="16"/>
 </signal>
 <signal name="DAC1">

Commit message: up
Parts:
- added CAN_TERM: can term, pinhead:1X02
- added ETH_5V: PTR1PAD1-13, testpad:P1-13
- moved S1 2.84 mm to (-38.1, 30.5)
- moved R5 2.54 mm to (-49.5, 26.7)
Connections:
- new net N$15: CAN_TERM.2, R5.2
- new net N$8: ETH_5V.TP, SV1.7
- net CANH: now also CAN_TERM.1; no longer R5.2
- net PWM1H: now also SV1.1
- net PWM1L: now also SV1.4
Routing:
- net SDI1_MODE: track 99.0 -> 128.7 mm, vias 3 -> 2
- net U1RX: track 44.7 -> 66.3 mm, vias 2 -> 3
- net VSS: track 243.8 -> 222.8 mm, vias 4 -> 8
- net PWM1H: track 40.3 -> 58.3 mm
- net SCK2: track 36.2 -> 23.2 mm
- net PWM1ER: track 28.9 -> 41.9 mm, vias 2 -> 0
- net PGD_C1TX: track 96.0 -> 83.9 mm, vias 3 -> 4
- net CANL: track 53.3 -> 63.8 mm
- net N$8: track 0.00 -> 10.2 mm
- net QEA2: track 20.2 -> 30.1 mm
- net AN0: track 30.8 -> 21.3 mm
- net GREEN_LED: track 58.1 -> 50.4 mm, vias 1 -> 2
- net SDI1: track 97.3 -> 89.7 mm
- net INDX2: track 18.9 -> 26.2 mm
- net IMU_CS: track 44.8 -> 51.3 mm
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