File: wfipic32host.brd (EAGLE design)
At the start: 95.2 x 42.9 mm, 64 parts, among them IC1 BMA490L, IC2 TCAN330GD, J1 MLE-105-01-G-DV, J2 MLE-105-01-G-DV, J3 MLE-105-01-G-DV, J4 MLE-105-01-G-DV, U1 PIC32MK0512MCJ048T-I/Y8XTQFP4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, U2 MAX6126B30

Commit message: up
Connections:
- net EXT_SW1 renamed DIS_CS
- net SDI1_MODE renamed DIS_RESET
- net SS1_OUT renamed DIS_MODE
Changed lines of the file:
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@@
 <via x="3.1242" y="32.385" extent="1-16" drill="0.35"/>
 </signal>
-<signal name="SDI1_MODE">
+<signal name="DIS_RESET">
 <contactref element="U1" pad="37"/>
 <contactref element="J1" pad="4"/>
@@
 <via x="23.3934" y="19.812" extent="1-16" drill="0.35"/>
 </signal>
-<signal name="SS1_OUT">
+<signal name="DIS_MODE">
 <contactref element="U1" pad="32"/>
 <contactref element="J1" pad="9"/>
@@
 <via x="26.4414" y="21.0312" extent="1-16" drill="0.35"/>
 </signal>
-<signal name="EXT_SW1">
+<signal name="DIS_CS">
 <contactref element="U1" pad="8"/>
 <contactref element="J1" pad="6"/>

Commit message: up
Parts:
- removed JP3: SIL, pinhead:1X02
- removed JP4: STB, pinhead:1X02
- added GND_POINTS: GND_TEST, pinhead:1X02
- added SJ1: can_shdn, jumper:SJ_2
- added SJ2: can_s, jumper:SJ_2
- moved J1 14.0 mm to (26.7, 38.1)
- moved C7 11.7 mm to (29.2, 20.3)
- moved J2 2.84 mm to (26.7, 47.0)
- moved J3 2.84 mm to (26.7, 55.9)
- moved C14 1.27 mm to (-16.5, 25.4)
- moved C15 1.27 mm to (-14.0, 25.4)
Connections:
- net N$12: now also SJ1.2; no longer JP4.2
- net N$13: now also SJ2.2; no longer JP3.2
- net VDD: now also SJ1.1, SJ2.1; no longer JP3.1, JP4.1
- net VSS: now also GND_POINTS.1, GND_POINTS.2, SJ1.3, SJ2.3
Routing:
- net VSS: track 222.8 -> 290.9 mm, vias 8 -> 4
- net DIS_RESET: track 128.7 -> 88.8 mm
- net SCK1: track 103.8 -> 141.3 mm, vias 1 -> 2
- net GREEN_LED: track 50.4 -> 83.3 mm, vias 2 -> 0
- net MCLR_SIG: track 71.0 -> 38.6 mm
- net N$12: track 18.6 -> 50.8 mm
- net PWM1ER: track 41.9 -> 18.6 mm, vias 0 -> 2
- net PWM1L: track 40.0 -> 63.1 mm
- net VDD: track 330.0 -> 307.3 mm, vias 5 -> 2
- net EXT_INT2: track 23.8 -> 39.9 mm
- net IMU_CS: track 51.3 -> 35.9 mm, vias 3 -> 4
- net PWM1H: track 58.3 -> 43.1 mm, vias 0 -> 2
- net PWM4ER: track 33.8 -> 47.3 mm
- net DIS_MODE: track 97.7 -> 84.1 mm
- net VREF+: track 98.1 -> 86.0 mm, vias 4 -> 5
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Other:
- board text added: "PIC32MK-CANFD HOST V1.7"
- board text removed: "PIC32MK-CANFD HOST V1.6"

Commit message: update PCB design
Parts:
- added UART_POINTS: UART_TEST, pinhead:1X02
- moved C15 2.84 mm to (-16.5, 26.7), turned to 90 degrees
- moved C14 2.84 mm to (-19.1, 26.7), turned to 90 degrees
- moved C18 2.54 mm to (-1.27, 27.9)
- moved C23 1.27 mm to (-1.27, 31.8)
- moved IC2 1.27 mm to (-7.62, 22.9)
- turned CAN_TERM to 270 degrees
Connections:
- net CANH renamed CAN_P
- net CANL renamed CAN_N
- net QEA2: now also SV2.9
- net QEB2: now also SV2.10
- net U1RX: now also UART_POINTS.1
- net U1TX: now also UART_POINTS.2
Routing:
- net QEA2: track 22.5 -> 105.0 mm, vias 2 -> 3
- net PGC_C1RX: track 80.4 -> 137.3 mm
- net QEB2: track 28.6 -> 85.4 mm, vias 2 -> 3
- net SCK1: track 141.3 -> 92.4 mm, vias 2 -> 3
- net VDD: track 307.3 -> 344.7 mm, vias 2 -> 7
- net SCK2: track 23.8 -> 50.8 mm, vias 2 -> 1
- net DIS_RESET: track 88.8 -> 114.2 mm
- net N$12: track 50.8 -> 26.0 mm
- net U1RX: track 59.5 -> 84.2 mm, vias 3 -> 2
- net GREEN_LED: track 83.3 -> 59.2 mm, vias 0 -> 1
- net PWM4ER: track 47.3 -> 33.8 mm
- net EXT_INT2: track 39.9 -> 26.4 mm
- net VSS: track 290.9 -> 279.0 mm, vias 4 -> 5
- net AVDD: track 55.3 -> 43.9 mm, vias 3 -> 2
- net RED_LED: track 34.9 -> 24.0 mm
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Other:
- board text added: "NSASPOOK@NSASPOOK.COM"

Commit message: up
Parts:
- moved C22 2.54 mm to (21.6, 20.3)
Routing:
- net VSS: track 279.0 -> 281.6 mm
- net VDD: track 344.7 -> 346.7 mm
- net DC_INPUT: track 34.5 -> 35.2 mm
Changed lines of the file:
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@@
 <attribute name="VALUE" x="15.24" y="17.78" size="1.27" layer="28" rot="MR0"/>
 </element>
-<element name="C22" library="rcl" library_urn="urn:adsk.eagle:library:334" package="C0805" package3d_urn="urn:adsk.eagle:package:23617/2" value="10uf" x="19.05" y="20.32" smashed="yes" rot="MR0">
-<attribute name="NAME" x="20.32" y="17.78" size="1.27" layer="26" rot="MR0"/>
-<attribute name="POPULARITY" value="63" x="19.05" y="20.32" size="1.778" layer="28" rot="MR0" display="off"/>
-<attribute name="SPICEPREFIX" value="C" x="19.05" y="20.32" size="1.778" layer="28" rot="MR0" display="off"/>
-<attribute name="VALUE" x="20.32" y="17.78" size="1.27" layer="28" rot="MR0"/>
+<element name="C22" library="rcl" library_urn="urn:adsk.eagle:library:334" package="C0805" package3d_urn="urn:adsk.eagle:package:23617/2" value="10uf" x="21.59" y="20.32" smashed="yes" rot="MR0">
+<attribute name="NAME" x="22.86" y="17.78" size="1.27" layer="26" rot="MR0"/>
+<attribute name="POPULARITY" value="63" x="21.59" y="20.32" size="1.778" layer="28" rot="MR0" display="off"/>
+<attribute name="SPICEPREFIX" value="C" x="21.59" y="20.32" size="1.778" layer="28" rot="MR0" display="off"/>
+<attribute name="VALUE" x="22.86" y="17.78" size="1.27" layer="28" rot="MR0"/>
 </element>
 <element name="JP6" library="pinhead" library_urn="urn:adsk.eagle:library:325" package="1X02" package3d_urn="urn:adsk.eagle:package:22435/2" value="DC12+" x="33.02" y="25.4" smashed="yes" rot="R90">
@@
 <wire x1="24.6888" y1="39.7764" x2="24.67" y2="39.7855" width="0.2032" layer="1"/>
 <wire x1="32.9946" y1="39.3192" x2="33.02" y2="39.37" width="0.2032" layer="1"/>
-<wire x1="17.4498" y1="22.86" x2="19.9644" y2="20.3454" width="0.2032" layer="16"/>
 <wire x1="16.51" y1="22.86" x2="17.4498" y2="22.86" width="0.2032" layer="16"/>
-<wire x1="19.9644" y1="20.3454" x2="20" y2="20.32" width="0.2032" layer="16"/>
+<wire x1="18.04249375" y1="23.52889375" x2="22.54" y2="20.32" width="0.2032" layer="16"/>
 <wire x1="22.6314" y1="20.3454" x2="28.194" y2="20.3454" width="0.2032" layer="1"/>
 <wire x1="20.1168" y1="22.86" x2="22.6314" y2="20.3454" width="0.2032" layer="1"/>
@@
 <wire x1="28.194" y1="20.3454" x2="28.26" y2="20.32" width="0.2032" layer="1"/>
 <wire x1="21.5646" y1="27.051" x2="21.5646" y2="30.7848" width="0.2032" layer="16"/>
-<wire x1="17.4498" y1="22.9362" x2="21.5646" y2="27.051" width="0.2032" layer="16"/>
+<wire x1="17.4498" y1="22.9362" x2="18.04249375" y2="23.52889375" width="0.2032" layer="16"/>
+<wire x1="18.04249375" y1="23.52889375" x2="21.5646" y2="27.051" width="0.2032" layer="16"/>
 <wire x1="21.5646" y1="30.7848" x2="21.59" y2="30.8" width="0.2032" layer="16"/>
 <wire x1="17.4498" y1="22.9362" x2="17.4498" y2="22.86" width="0.2032" layer="16"/>
@@
 <wire x1="13.0302" y1="20.3454" x2="13.02" y2="20.32" width="0.2032" layer="16"/>
 <wire x1="13.9446" y1="22.86" x2="13.97" y2="22.86" width="0.2032" layer="16"/>
-<wire x1="16.6878" y1="20.3454" x2="18.0594" y2="20.3454" width="0.2032" layer="16"/>
+<wire x1="16.6878" y1="20.3454" x2="20.5994" y2="20.3454" width="0.2032" layer="16"/>
 <wire x1="14.2494" y1="22.7838" x2="16.6878" y2="20.3454" width="0.2032" layer="16"/>
 <wire x1="14.0208" y1="22.7838" x2="14.2494" y2="22.7838" width="0.2032" layer="16"/>
-<wire x1="18.0594" y1="20.3454" x2="18.1" y2="20.32" width="0.2032" layer="16"/>
+<wire x1="20.5994" y1="20.3454" x2="20.64" y2="20.32" width="0.2032" layer="16"/>
 <wire x1="14.0208" y1="22.7838" x2="13.97" y2="22.86" width="0.2032" layer="16"/>
 <wire x1="30.099" y1="23.241" x2="30.099" y2="20.3454" width="0.2032" layer="1"/>
@@
 <wire x1="11.43" y1="22.86" x2="9.906" y2="21.336" width="0.3048" layer="16"/>
 <wire x1="9.906" y1="20.3454" x2="9.84" y2="20.32" width="0.3048" layer="16"/>
-<wire x1="13.7922" y1="19.2024" x2="14.859" y2="20.2692" width="0.3048" layer="16"/>
-<wire x1="11.2014" y1="19.2024" x2="13.7922" y2="19.2024" width="0.3048" layer="16"/>
+<wire x1="14.92" y1="20.32" x2="14.92" y2="19.2024" width="0.3048" layer="16"/>
+<wire x1="11.2014" y1="19.2024" x2="14.92" y2="19.2024" width="0.3048" layer="16"/>
 <wire x1="10.0584" y1="20.3454" x2="11.2014" y2="19.2024" width="0.3048" layer="16"/>
-<wire x1="14.859" y1="20.2692" x2="14.92" y2="20.32" width="0.3048" layer="16"/>
 <wire x1="10.0584" y1="20.3454" x2="9.84" y2="20.32" width="0.3048" layer="16"/>
 <wire x1="32.9946" y1="32.766" x2="32.9946" y2="33.147" width="0.3048" layer="16"/>
