File: wfipic32host.sch (EAGLE design)
At the start: 40 parts, among them IC1 BMA490L, IC2 TCAN330GD, J1 MLE-105-01-G-DV, J2 MLE-105-01-G-DV, J3 MLE-105-01-G-DV, J4 MLE-105-01-G-DV, U1 PIC32MK0512MCJ048T-I/Y8XTQFP4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, U2 MAX6126B30

Commit message: up
Parts:
- added C14, C16: 10uf, rcl:C-USC0805
- added C15, C17: 0.1uf, rcl:C-USC0805
- added SV1: ETH1, con-lstb:MA07-1
- added SV4, SV5: ETHG, con-lstb:MA03-1
- JP3: value RESET_JMP -> SIL
- JP4: value RESET_JMP -> STB
Connections:
- net U1RX: now also SV1.3
- net U1TX: now also SV1.2
- net VDD: now also C14.1, C15.1, C16.1, C17.1, SV1.6
- net VSS: now also C14.2, C15.2, C16.2, C17.2, SV1.5, SV4.1, SV4.2, SV4.3, SV5.1, SV5.2, SV5.3

Commit message: up
Parts:
- added 3.3VDC: 3.3 Vreg, linear:7805TV
- added C18, C19, C20: 0.1uf, rcl:C-USC0805
- added C21, C22: 10uf, rcl:C-USC0805
- added JP6: DC5+, pinhead:PINHD-1X2
- added OS1: OSC-OE-CFPS-32, IQD-Frequency-Products:OSC-OE-CFPS-32
- added R6: 0 ohm fuse, rcl:R-US_M1206
- renumbered REFCLK2 to GLED
Connections:
- removed net N$8: GLED.TP, U1.OA5IN+/AN24/CVD24/C5IN1+/C5IN3-/RPA4/RA4
- new net DC_IN: JP6.2, R6.2
- new net DC_INPUT: 3.3VDC.VI, C20.1, C21.1, R6.1
- new net OSC_MCU: OS1.OUT, U1.OSCI/CLKI/AN49/CVD49/RPC12/RC12
- net GREEN_LED: now also GLED.TP, U1.OA5IN+/AN24/CVD24/C5IN1+/C5IN3-/RPA4/RA4; no longer U1.OSCI/CLKI/AN49/CVD49/RPC12/RC12
- net VDD: now also 3.3VDC.VO, C18.1, C19.1, C22.1, OS1.CON, OS1.VDD
- net VSS: now also 3.3VDC.GND, C18.2, C19.2, C20.2, C21.2, C22.2, JP6.1, OS1.VSS

Commit message: up
Connections:
- net VDD: now also IC2.VCC; no longer IC2.GND
- net VSS: now also IC2.GND; no longer IC2.VCC
Changed lines of the file:
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@@
 <part name="VSS22" library="supply1" library_urn="urn:adsk.eagle:library:371" deviceset="VSS" device=""/>
 <part name="IC2" library="TCAN330GD" deviceset="TCAN330GD" device=""/>
-<part name="VSS23" library="supply1" library_urn="urn:adsk.eagle:library:371" deviceset="VSS" device=""/>
-<part name="VDD3" library="supply1" library_urn="urn:adsk.eagle:library:371" deviceset="VDD" device=""/>
 <part name="JP3" library="pinhead" library_urn="urn:adsk.eagle:library:325" deviceset="PINHD-1X2" device="" package3d_urn="urn:adsk.eagle:package:22435/2" value="SIL"/>
 <part name="JP4" library="pinhead" library_urn="urn:adsk.eagle:library:325" deviceset="PINHD-1X2" device="" package3d_urn="urn:adsk.eagle:package:22435/2" value="STB"/>
@@
 <part name="VSS37" library="supply1" library_urn="urn:adsk.eagle:library:371" deviceset="VSS" device=""/>
 <part name="R6" library="rcl" library_urn="urn:adsk.eagle:library:334" deviceset="R-US_" device="M1206" package3d_urn="urn:adsk.eagle:package:23566/2" value="0 ohm fuse"/>
+<part name="VSS38" library="supply1" library_urn="urn:adsk.eagle:library:371" deviceset="VSS" device=""/>
+<part name="VDD3" library="supply1" library_urn="urn:adsk.eagle:library:371" deviceset="VDD" device=""/>
 </parts>
 <sheets>
@@
 <attribute name="VALUE" x="-29.21" y="147.32" size="1.778" layer="96" align="center-left"/>
 </instance>
-<instance part="VSS23" gate="G$1" x="-58.42" y="134.62" smashed="yes">
-<attribute name="VALUE" x="-60.96" y="129.54" size="1.778" layer="96" rot="R90"/>
-</instance>
-<instance part="VDD3" gate="G$1" x="-58.42" y="142.24" smashed="yes">
-<attribute name="VALUE" x="-60.96" y="139.7" size="1.778" layer="96" rot="R90"/>
-</instance>
 <instance part="JP3" gate="G$1" x="-7.62" y="152.4" smashed="yes">
 <attribute name="NAME" x="-13.97" y="158.115" size="1.778" layer="95"/>
@@
 <attribute name="NAME" x="140.97" y="-37.0586" size="1.778" layer="95" rot="R180"/>
 <attribute name="VALUE" x="140.97" y="-32.258" size="1.778" layer="96" rot="R180"/>
+</instance>
+<instance part="VSS38" gate="G$1" x="-58.42" y="142.24" smashed="yes" rot="R180">
+<attribute name="VALUE" x="-55.88" y="147.32" size="1.778" layer="96" rot="R270"/>
+</instance>
+<instance part="VDD3" gate="G$1" x="-58.42" y="134.62" smashed="yes" rot="R180">
+<attribute name="VALUE" x="-55.88" y="137.16" size="1.778" layer="96" rot="R270"/>
 </instance>
 </instances>
@@
 </segment>
 <segment>
-<pinref part="IC2" gate="G$1" pin="GND"/>
-<wire x1="-53.34" y1="139.7" x2="-58.42" y2="139.7" width="0.1524" layer="91"/>
-<pinref part="VDD3" gate="G$1" pin="VDD"/>
-<junction x="-53.34" y="139.7"/>
-<junction x="-58.42" y="139.7"/>
-</segment>
-<segment>
 <wire x1="-22.86" y1="154.94" x2="-10.16" y2="154.94" width="0.1524" layer="91"/>
 <pinref part="JP3" gate="G$1" pin="1"/>
@@
 <wire x1="180.34" y1="-35.56" x2="187.96" y2="-35.56" width="0.1524" layer="91"/>
 <pinref part="C22" gate="G$1" pin="1"/>
+</segment>
+<segment>
+<pinref part="IC2" gate="G$1" pin="VCC"/>
+<wire x1="-53.34" y1="137.16" x2="-58.42" y2="137.16" width="0.1524" layer="91"/>
+<junction x="-53.34" y="137.16"/>
+<pinref part="VDD3" gate="G$1" pin="VDD"/>
+<junction x="-58.42" y="137.16"/>
 </segment>
 </net>
@@
 <junction x="-38.1" y="-27.94"/>
 <junction x="-30.48" y="-27.94"/>
-</segment>
-<segment>
-<pinref part="IC2" gate="G$1" pin="VCC"/>
-<wire x1="-53.34" y1="137.16" x2="-58.42" y2="137.16" width="0.1524" layer="91"/>
-<pinref part="VSS23" gate="G$1" pin="VSS"/>
-<junction x="-53.34" y="137.16"/>
-<junction x="-58.42" y="137.16"/>
 </segment>
 <segment>
@@
 <junction x="124.46" y="-50.8"/>
 </segment>
+<segment>
+<pinref part="IC2" gate="G$1" pin="GND"/>
+<wire x1="-53.34" y1="139.7" x2="-58.42" y2="139.7" width="0.1524" layer="91"/>
+<junction x="-53.34" y="139.7"/>
+<pinref part="VSS38" gate="G$1" pin="VSS"/>
+<junction x="-58.42" y="139.7"/>
+</segment>
 </net>

Commit message: up
Parts:
- added SV2: GLCD, con-lstb:MA10-1
Connections:
- net EXT_SW1: now also SV2.5
- net SCK1: now also SV2.3
- net SDI1: now also SV2.1
- net SDI1_MODE: now also SV2.6
- net SDO1: now also SV2.2
- net SS1_OUT: now also SV2.4
- net VDD: now also SV2.7
- net VSS: now also SV2.8
Changed lines of the file:
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@@
 <part name="VSS38" library="supply1" library_urn="urn:adsk.eagle:library:371" deviceset="VSS" device=""/>
 <part name="VDD3" library="supply1" library_urn="urn:adsk.eagle:library:371" deviceset="VDD" device=""/>
+<part name="SV2" library="con-lstb" library_urn="urn:adsk.eagle:library:162" deviceset="MA10-1" device="" package3d_urn="urn:adsk.eagle:package:8346/1" value="GLCD"/>
+<part name="VSS23" library="supply1" library_urn="urn:adsk.eagle:library:371" deviceset="VSS" device=""/>
+<part name="VDD15" library="supply1" library_urn="urn:adsk.eagle:library:371" deviceset="VDD" device=""/>
 </parts>
 <sheets>
@@
 <instance part="VDD3" gate="G$1" x="-58.42" y="134.62" smashed="yes" rot="R180">
 <attribute name="VALUE" x="-55.88" y="137.16" size="1.778" layer="96" rot="R270"/>
+</instance>
+<instance part="SV2" gate="1" x="-106.68" y="5.08" smashed="yes">
+<attribute name="VALUE" x="-107.95" y="-10.16" size="1.778" layer="96"/>
+<attribute name="NAME" x="-107.95" y="21.082" size="1.778" layer="95"/>
+</instance>
+<instance part="VSS23" gate="G$1" x="-86.36" y="15.24" smashed="yes" rot="R180">
+<attribute name="VALUE" x="-88.9" y="17.78" size="1.778" layer="96"/>
+</instance>
+<instance part="VDD15" gate="G$1" x="-81.28" y="12.7" smashed="yes">
+<attribute name="VALUE" x="-73.66" y="12.7" size="1.778" layer="96" rot="R180"/>
 </instance>
 </instances>
@@
 <pinref part="VDD3" gate="G$1" pin="VDD"/>
 <junction x="-58.42" y="137.16"/>
+</segment>
+<segment>
+<pinref part="SV2" gate="1" pin="7"/>
+<wire x1="-99.06" y1="10.16" x2="-81.28" y2="10.16" width="0.1524" layer="91"/>
+<pinref part="VDD15" gate="G$1" pin="VDD"/>
 </segment>
 </net>
@@
 <junction x="-58.42" y="139.7"/>
 </segment>
+<segment>
+<pinref part="SV2" gate="1" pin="8"/>
+<wire x1="-99.06" y1="12.7" x2="-86.36" y2="12.7" width="0.1524" layer="91"/>
+<pinref part="VSS23" gate="G$1" pin="VSS"/>
+</segment>
 </net>
 <net name="AVDD" class="0">
@@
 <junction x="205.74" y="121.92"/>
 </segment>
+<segment>
+<wire x1="-99.06" y1="7.62" x2="-86.36" y2="7.62" width="0.1524" layer="91"/>
+<pinref part="SV2" gate="1" pin="6"/>
+<label x="-83.82" y="7.62" size="1.778" layer="95"/>
+</segment>
 </net>
 <net name="SDI1" class="0">
@@
 <label x="147.32" y="124.46" size="1.778" layer="95"/>
 </segment>
+<segment>
+<wire x1="-86.36" y1="-5.08" x2="-99.06" y2="-5.08" width="0.1524" layer="91"/>
+<pinref part="SV2" gate="1" pin="1"/>
+<label x="-83.82" y="-5.08" size="1.778" layer="95"/>
+</segment>
 </net>
 <net name="SDO1" class="0">
@@
 <junction x="170.18" y="127"/>
 </segment>
+<segment>
+<wire x1="-99.06" y1="-2.54" x2="-86.36" y2="-2.54" width="0.1524" layer="91"/>
+<pinref part="SV2" gate="1" pin="2"/>
+<label x="-86.36" y="-2.54" size="1.778" layer="95"/>
+</segment>
 </net>
 <net name="SS1_OUT" class="0">
@@
 <junction x="157.48" y="129.54"/>
 </segment>
+<segment>
+<wire x1="-99.06" y1="2.54" x2="-86.36" y2="2.54" width="0.1524" layer="91"/>
+<pinref part="SV2" gate="1" pin="4"/>
+<label x="-86.36" y="2.54" size="1.778" layer="95"/>
+</segment>
 </net>
 <net name="EXT_SW1" class="0">
@@
 <junction x="193.04" y="124.46"/>
 <junction x="205.74" y="124.46"/>
+</segment>
+<segment>
+<wire x1="-86.36" y1="5.08" x2="-99.06" y2="5.08" width="0.1524" layer="91"/>
+<pinref part="SV2" gate="1" pin="5"/>
+<label x="-83.82" y="5.08" size="1.778" layer="95"/>
 </segment>
 </net>
@@
 <junction x="205.74" y="127"/>
 </segment>
-</net>
+<segment>
+<wire x1="-99.06" y1="0" x2="-86.36" y2="0" width="0.1524" layer="91"/>
+<pinref part="SV2" gate="1" pin="3"/>
+<label x="-86.36" y="0" size="1.778" layer="95"/>
+</segment>
+</net>

Commit message: up
Parts:
- added 3.3VTP, GND_TP, OSCI, VREF_TP: PTR1PAD1-13, testpad:PTR1PAD1-13
- added C23: 10uf, rcl:C-USC0805
- JP6: value DC5+ -> DC12+
Connections:
- net AVDD: now also C23.1
- net OSC_MCU: now also OSCI.TP
- net VDD: now also 3.3VTP.TP
- net VREF+: now also VREF_TP.TP
- net VSS: now also C23.2, GND_TP.TP
Changed lines of the file:
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@@
 <part name="VSS35" library="supply1" library_urn="urn:adsk.eagle:library:371" deviceset="VSS" device=""/>
 <part name="VSS36" library="supply1" library_urn="urn:adsk.eagle:library:371" deviceset="VSS" device=""/>
-<part name="JP6" library="pinhead" library_urn="urn:adsk.eagle:library:325" deviceset="PINHD-1X2" device="" package3d_urn="urn:adsk.eagle:package:22435/2" value="DC5+"/>
+<part name="JP6" library="pinhead" library_urn="urn:adsk.eagle:library:325" deviceset="PINHD-1X2" device="" package3d_urn="urn:adsk.eagle:package:22435/2" value="DC12+"/>
 <part name="VSS37" library="supply1" library_urn="urn:adsk.eagle:library:371" deviceset="VSS" device=""/>
 <part name="R6" library="rcl" library_urn="urn:adsk.eagle:library:334" deviceset="R-US_" device="M1206" package3d_urn="urn:adsk.eagle:package:23566/2" value="0 ohm fuse"/>
@@
 <part name="VSS23" library="supply1" library_urn="urn:adsk.eagle:library:371" deviceset="VSS" device=""/>
 <part name="VDD15" library="supply1" library_urn="urn:adsk.eagle:library:371" deviceset="VDD" device=""/>
+<part name="OSCI" library="testpad" library_urn="urn:adsk.eagle:library:385" deviceset="PTR1" device="PAD1-13" package3d_urn="urn:adsk.eagle:package:27946/1"/>
+<part name="3.3VTP" library="testpad" library_urn="urn:adsk.eagle:library:385" deviceset="PTR1" device="PAD1-13" package3d_urn="urn:adsk.eagle:package:27946/1"/>
+<part name="GND_TP" library="testpad" library_urn="urn:adsk.eagle:library:385" deviceset="PTR1" device="PAD1-13" package3d_urn="urn:adsk.eagle:package:27946/1"/>
+<part name="VSS39" library="supply1" library_urn="urn:adsk.eagle:library:371" deviceset="VSS" device=""/>
+<part name="VREF_TP" library="testpad" library_urn="urn:adsk.eagle:library:385" deviceset="PTR1" device="PAD1-13" package3d_urn="urn:adsk.eagle:package:27946/1"/>
+<part name="C23" library="rcl" library_urn="urn:adsk.eagle:library:334" deviceset="C-US" device="C0805" package3d_urn="urn:adsk.eagle:package:23617/2" value="10uf"/>
+<part name="VSS40" library="supply1" library_urn="urn:adsk.eagle:library:371" deviceset="VSS" device=""/>
 </parts>
 <sheets>
@@
 <instance part="VDD15" gate="G$1" x="-81.28" y="12.7" smashed="yes">
 <attribute name="VALUE" x="-73.66" y="12.7" size="1.778" layer="96" rot="R180"/>
+</instance>
+<instance part="OSCI" gate="G$1" x="254" y="-30.48" smashed="yes" rot="R180">
+<attribute name="NAME" x="255.016" y="-24.13" size="1.778" layer="95" rot="R270"/>
+<attribute name="TP_SIGNAL_NAME" x="252.73" y="-27.94" size="1.778" layer="97" rot="R180"/>
+</instance>
+<instance part="3.3VTP" gate="G$1" x="187.96" y="-33.02" smashed="yes" rot="R180">
+<attribute name="NAME" x="188.976" y="-26.67" size="1.778" layer="95" rot="R270"/>
+<attribute name="TP_SIGNAL_NAME" x="186.69" y="-30.48" size="1.778" layer="97" rot="R180"/>
+</instance>
+<instance part="GND_TP" gate="G$1" x="198.12" y="-33.02" smashed="yes" rot="R180">
+<attribute name="NAME" x="199.136" y="-26.67" size="1.778" layer="95" rot="R270"/>
+<attribute name="TP_SIGNAL_NAME" x="196.85" y="-30.48" size="1.778" layer="97" rot="R180"/>
+</instance>
+<instance part="VSS39" gate="G$1" x="198.12" y="-38.1" smashed="yes">
+<attribute name="VALUE" x="195.58" y="-43.18" size="1.778" layer="96" rot="R90"/>
+</instance>
+<instance part="VREF_TP" gate="G$1" x="137.16" y="-2.54" smashed="yes" rot="R180">
+<attribute name="NAME" x="138.176" y="3.81" size="1.778" layer="95" rot="R270"/>
+<attribute name="TP_SIGNAL_NAME" x="135.89" y="0" size="1.778" layer="97" rot="R180"/>
+</instance>
+<instance part="C23" gate="G$1" x="30.48" y="144.78" smashed="yes">
+<attribute name="NAME" x="31.496" y="145.415" size="1.778" layer="95"/>
+<attribute name="VALUE" x="31.496" y="140.589" size="1.778" layer="96"/>
+</instance>
+<instance part="VSS40" gate="G$1" x="30.48" y="137.16" smashed="yes">
+<attribute name="VALUE" x="27.94" y="132.08" size="1.778" layer="96" rot="R90"/>
 </instance>
 </instances>
@@
 <wire x1="180.34" y1="-35.56" x2="187.96" y2="-35.56" width="0.1524" layer="91"/>
 <pinref part="C22" gate="G$1" pin="1"/>
+<pinref part="3.3VTP" gate="G$1" pin="TP"/>
+<junction x="187.96" y="-35.56"/>
 </segment>
 <segment>
@@
 <wire x1="-99.06" y1="10.16" x2="-81.28" y2="10.16" width="0.1524" layer="91"/>
 <pinref part="VDD15" gate="G$1" pin="VDD"/>
+<junction x="-81.28" y="10.16"/>
+<junction x="-99.06" y="10.16"/>
 </segment>
 </net>
@@
 <wire x1="-99.06" y1="12.7" x2="-86.36" y2="12.7" width="0.1524" layer="91"/>
 <pinref part="VSS23" gate="G$1" pin="VSS"/>
+<junction x="-86.36" y="12.7"/>
+<junction x="-99.06" y="12.7"/>
+</segment>
+<segment>
+<pinref part="GND_TP" gate="G$1" pin="TP"/>
+<pinref part="VSS39" gate="G$1" pin="VSS"/>
+</segment>
+<segment>
+<pinref part="C23" gate="G$1" pin="2"/>
+<pinref part="VSS40" gate="G$1" pin="VSS"/>
 </segment>
 </net>
@@
 <label x="33.02" y="142.24" size="1.778" layer="95"/>
 <wire x1="22.86" y1="147.32" x2="30.48" y2="147.32" width="0.1524" layer="91"/>
+<pinref part="C23" gate="G$1" pin="1"/>
 </segment>
 <segment>
@@
 <label x="241.3" y="-38.1" size="1.778" layer="95"/>
 <junction x="254" y="-33.02"/>
+<pinref part="OSCI" gate="G$1" pin="TP"/>
 </segment>
 </net>
@@
 <pinref part="SV2" gate="1" pin="6"/>
 <label x="-83.82" y="7.62" size="1.778" layer="95"/>
+<junction x="-86.36" y="7.62"/>
+<junction x="-99.06" y="7.62"/>
 </segment>
 </net>
@@
 <pinref part="SV2" gate="1" pin="1"/>
 <label x="-83.82" y="-5.08" size="1.778" layer="95"/>
+<junction x="-86.36" y="-5.08"/>
+<junction x="-99.06" y="-5.08"/>
 </segment>
 </net>
@@
 <pinref part="SV2" gate="1" pin="2"/>
 <label x="-86.36" y="-2.54" size="1.778" layer="95"/>
+<junction x="-86.36" y="-2.54"/>
+<junction x="-99.06" y="-2.54"/>
 </segment>
 </net>
@@
 <pinref part="SV2" gate="1" pin="4"/>
 <label x="-86.36" y="2.54" size="1.778" layer="95"/>
+<junction x="-86.36" y="2.54"/>
+<junction x="-99.06" y="2.54"/>
 </segment>
 </net>
@@
 <pinref part="SV2" gate="1" pin="5"/>
 <label x="-83.82" y="5.08" size="1.778" layer="95"/>
+<junction x="-86.36" y="5.08"/>
+<junction x="-99.06" y="5.08"/>
 </segment>
 </net>
@@
 <junction x="137.16" y="-17.78"/>
 <label x="139.7" y="-20.32" size="1.778" layer="95"/>
+<pinref part="VREF_TP" gate="G$1" pin="TP"/>
+<junction x="137.16" y="-5.08"/>
 </segment>
 </net>
@@
 <pinref part="SV2" gate="1" pin="3"/>
 <label x="-86.36" y="0" size="1.778" layer="95"/>
-</segment>
-</net>
+<junction x="-86.36" y="0"/>
+<junction x="-99.06" y="0"/>
+</segment>
+</net>

Commit message: up
Parts:
- added CAN_TERM: can term, pinhead:PINHD-1X2
- added ETH_5V: PTR1PAD1-13, testpad:PTR1PAD1-13
Connections:
- new net N$15: CAN_TERM.2, R5.2
- new net N$8: ETH_5V.TP, SV1.7
- net CANH: now also CAN_TERM.1; no longer R5.2
- net PWM1H: now also SV1.1
- net PWM1L: now also SV1.4
Changed lines of the file:
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@@
 <class number="1" name="icurrent" width="0.3048" drill="0">
+</class>
+<class number="2" name="ncurrent" width="0.2032" drill="0">
 </class>
 </classes>
@@
 <part name="C23" library="rcl" library_urn="urn:adsk.eagle:library:334" deviceset="C-US" device="C0805" package3d_urn="urn:adsk.eagle:package:23617/2" value="10uf"/>
 <part name="VSS40" library="supply1" library_urn="urn:adsk.eagle:library:371" deviceset="VSS" device=""/>
+<part name="ETH_5V" library="testpad" library_urn="urn:adsk.eagle:library:385" deviceset="PTR1" device="PAD1-13" package3d_urn="urn:adsk.eagle:package:27946/1"/>
+<part name="CAN_TERM" library="pinhead" library_urn="urn:adsk.eagle:library:325" deviceset="PINHD-1X2" device="" package3d_urn="urn:adsk.eagle:package:22435/2" value="can term"/>
 </parts>
 <sheets>
@@
 <attribute name="VALUE" x="27.94" y="132.08" size="1.778" layer="96" rot="R90"/>
 </instance>
+<instance part="ETH_5V" gate="G$1" x="-73.66" y="73.66" smashed="yes" rot="R180">
+<attribute name="NAME" x="-72.644" y="80.01" size="1.778" layer="95" rot="R270"/>
+<attribute name="TP_SIGNAL_NAME" x="-74.93" y="76.2" size="1.778" layer="97" rot="R180"/>
+</instance>
+<instance part="CAN_TERM" gate="G$1" x="10.16" y="152.4" smashed="yes">
+<attribute name="NAME" x="3.81" y="158.115" size="1.778" layer="95"/>
+<attribute name="VALUE" x="3.81" y="147.32" size="1.778" layer="96"/>
+</instance>
 </instances>
 <busses>
 </busses>
 <nets>
-<net name="VDD" class="0">
+<net name="VDD" class="2">
 <segment>
 <wire x1="5.08" y1="132.08" x2="10.16" y2="132.08" width="0.1524" layer="91"/>
@@
 </segment>
 </net>
-<net name="VSS" class="0">
+<net name="VSS" class="2">
 <segment>
 <wire x1="7.62" y1="124.46" x2="10.16" y2="124.46" width="0.1524" layer="91"/>
@@
 </segment>
 </net>
-<net name="AVDD" class="0">
+<net name="AVDD" class="2">
 <segment>
 <pinref part="L1" gate="G$1" pin="1"/>
@@
 <junction x="157.48" y="-7.62"/>
 </segment>
+<segment>
+<wire x1="-60.96" y1="63.5" x2="-73.66" y2="63.5" width="0.1524" layer="91"/>
+<pinref part="SV1" gate="1" pin="4"/>
+<label x="-66.04" y="63.5" size="1.778" layer="95"/>
+<junction x="-73.66" y="63.5"/>
+<junction x="-60.96" y="63.5"/>
+</segment>
 </net>
 <net name="PWM1H" class="0">
@@
 <junction x="170.18" y="-5.08"/>
 <junction x="170.18" y="-5.08"/>
+</segment>
+<segment>
+<wire x1="-60.96" y1="55.88" x2="-73.66" y2="55.88" width="0.1524" layer="91"/>
+<pinref part="SV1" gate="1" pin="1"/>
+<label x="-66.04" y="55.88" size="1.778" layer="95"/>
+<junction x="-73.66" y="55.88"/>
+<junction x="-60.96" y="55.88"/>
 </segment>
 </net>
@@
 <junction x="-25.4" y="139.7"/>
 <junction x="-15.24" y="139.7"/>
-<pinref part="R5" gate="G$1" pin="2"/>
-<wire x1="-5.08" y1="142.24" x2="-15.24" y2="142.24" width="0.1524" layer="91"/>
-<wire x1="-15.24" y1="142.24" x2="-15.24" y2="139.7" width="0.1524" layer="91"/>
-<junction x="-5.08" y="142.24"/>
+<pinref part="CAN_TERM" gate="G$1" pin="1"/>
+<wire x1="7.62" y1="154.94" x2="-2.54" y2="154.94" width="0.1524" layer="91"/>
+<wire x1="-2.54" y1="154.94" x2="-2.54" y2="147.32" width="0.1524" layer="91"/>
+<wire x1="-2.54" y1="147.32" x2="-15.24" y2="147.32" width="0.1524" layer="91"/>
+<wire x1="-15.24" y1="147.32" x2="-15.24" y2="139.7" width="0.1524" layer="91"/>
+<junction x="7.62" y="154.94"/>
 </segment>
 <segment>
@@
 </segment>
 </net>
+<net name="N$8" class="0">
+<segment>
+<pinref part="SV1" gate="1" pin="7"/>
+<pinref part="ETH_5V" gate="G$1" pin="TP"/>
+<junction x="-73.66" y="71.12"/>
+</segment>
+</net>
+<net name="N$15" class="0">
+<segment>
+<pinref part="CAN_TERM" gate="G$1" pin="2"/>
+<wire x1="7.62" y1="152.4" x2="0" y2="152.4" width="0.1524" layer="91"/>
+<wire x1="0" y1="152.4" x2="0" y2="142.24" width="0.1524" layer="91"/>
+<pinref part="R5" gate="G$1" pin="2"/>
+<wire x1="0" y1="142.24" x2="-5.08" y2="142.24" width="0.1524" layer="91"/>
+<junction x="-5.08" y="142.24"/>
+<junction x="7.62" y="152.4"/>
+</segment>
+</net>

Commit message: up
Connections:
- net EXT_SW1 renamed DIS_CS
- net SDI1_MODE renamed DIS_RESET
- net SS1_OUT renamed DIS_MODE
Changed lines of the file:
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@@
 </segment>
 </net>
-<net name="SDI1_MODE" class="0">
+<net name="DIS_RESET" class="0">
 <segment>
 <pinref part="U1" gate="A" pin="TMS/OA5IN-/AN27/CVD27/LVDIN/C5IN1-/RPB9/RB9"/>
@@
 </segment>
 </net>
-<net name="SS1_OUT" class="0">
+<net name="DIS_MODE" class="0">
 <segment>
 <pinref part="U1" gate="A" pin="PGC2/RPB6/SCL1/RB6"/>
@@
 </segment>
 </net>
-<net name="EXT_SW1" class="0">
+<net name="DIS_CS" class="0">
 <segment>
 <pinref part="U1" gate="A" pin="AN9/CVD9/RPA11/FLT14/RA11"/>
