File: wfipic32host.sch (EAGLE design)
At the start: 64 parts, among them IC1 BMA490L, IC2 TCAN330GD, J1 MLE-105-01-G-DV, J2 MLE-105-01-G-DV, J3 MLE-105-01-G-DV, J4 MLE-105-01-G-DV, U1 PIC32MK0512MCJ048T-I/Y8XTQFP4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, U2 MAX6126B30

Commit message: up
Parts:
- removed JP3: SIL, pinhead:PINHD-1X2
- removed JP4: STB, pinhead:PINHD-1X2
- added GND_POINTS: GND_TEST, pinhead:PINHD-1X2
- added SJ1: can_shdn, jumper:SJ2W
- added SJ2: can_s, jumper:SJ2W
Connections:
- net N$12: now also SJ1.2; no longer JP4.2
- net N$13: now also SJ2.2; no longer JP3.2
- net VDD: now also SJ1.1, SJ2.1; no longer JP3.1, JP4.1
- net VSS: now also GND_POINTS.1, GND_POINTS.2, SJ1.3, SJ2.3
Changed lines of the file:
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@@
 <part name="VSS22" library="supply1" library_urn="urn:adsk.eagle:library:371" deviceset="VSS" device=""/>
 <part name="IC2" library="TCAN330GD" deviceset="TCAN330GD" device=""/>
-<part name="JP3" library="pinhead" library_urn="urn:adsk.eagle:library:325" deviceset="PINHD-1X2" device="" package3d_urn="urn:adsk.eagle:package:22435/2" value="SIL"/>
-<part name="JP4" library="pinhead" library_urn="urn:adsk.eagle:library:325" deviceset="PINHD-1X2" device="" package3d_urn="urn:adsk.eagle:package:22435/2" value="STB"/>
 <part name="S1" library="JS202011SCQN_fixed" deviceset="JS202011SCQN" device=""/>
 <part name="JP5" library="pinhead" library_urn="urn:adsk.eagle:library:325" deviceset="PINHD-1X4" device="/90" package3d_urn="urn:adsk.eagle:package:22404/2" value="CAN-FD"/>
@@
 <part name="ETH_5V" library="testpad" library_urn="urn:adsk.eagle:library:385" deviceset="PTR1" device="PAD1-13" package3d_urn="urn:adsk.eagle:package:27946/1"/>
 <part name="CAN_TERM" library="pinhead" library_urn="urn:adsk.eagle:library:325" deviceset="PINHD-1X2" device="" package3d_urn="urn:adsk.eagle:package:22435/2" value="can term"/>
+<part name="SJ1" library="jumper" library_urn="urn:adsk.eagle:library:252" deviceset="SJ2W" device="" package3d_urn="urn:adsk.eagle:package:15474/1" value="can_shdn"/>
+<part name="SJ2" library="jumper" library_urn="urn:adsk.eagle:library:252" deviceset="SJ2W" device="" package3d_urn="urn:adsk.eagle:package:15474/1" value="can_s"/>
+<part name="VSS41" library="supply1" library_urn="urn:adsk.eagle:library:371" deviceset="VSS" device=""/>
+<part name="VSS42" library="supply1" library_urn="urn:adsk.eagle:library:371" deviceset="VSS" device=""/>
+<part name="GND_POINTS" library="pinhead" library_urn="urn:adsk.eagle:library:325" deviceset="PINHD-1X2" device="" package3d_urn="urn:adsk.eagle:package:22435/2" value="GND_TEST"/>
+<part name="VSS43" library="supply1" library_urn="urn:adsk.eagle:library:371" deviceset="VSS" device=""/>
 </parts>
 <sheets>
@@
 <attribute name="VALUE" x="-29.21" y="147.32" size="1.778" layer="96" align="center-left"/>
 </instance>
-<instance part="JP3" gate="G$1" x="-7.62" y="152.4" smashed="yes">
-<attribute name="NAME" x="-13.97" y="158.115" size="1.778" layer="95"/>
-<attribute name="VALUE" x="-13.97" y="147.32" size="1.778" layer="96"/>
-</instance>
-<instance part="JP4" gate="G$1" x="-7.62" y="121.92" smashed="yes">
-<attribute name="NAME" x="-13.97" y="127.635" size="1.778" layer="95"/>
-<attribute name="VALUE" x="-13.97" y="116.84" size="1.778" layer="96"/>
-</instance>
 <instance part="S1" gate="G$1" x="-83.82" y="137.16" smashed="yes">
 <attribute name="NAME" x="-99.0822" y="139.7037" size="1.27185" layer="95"/>
@@
 <attribute name="NAME" x="3.81" y="158.115" size="1.778" layer="95"/>
 <attribute name="VALUE" x="3.81" y="147.32" size="1.778" layer="96"/>
+</instance>
+<instance part="SJ1" gate="G$1" x="-7.62" y="119.38" smashed="yes">
+<attribute name="NAME" x="-2.54" y="117.221" size="1.778" layer="95"/>
+<attribute name="VALUE" x="-15.24" y="125.095" size="1.778" layer="96"/>
+</instance>
+<instance part="SJ2" gate="G$1" x="-10.16" y="157.48" smashed="yes">
+<attribute name="NAME" x="-7.62" y="157.861" size="1.778" layer="95"/>
+<attribute name="VALUE" x="-15.24" y="163.195" size="1.778" layer="96"/>
+</instance>
+<instance part="VSS41" gate="G$1" x="-7.62" y="111.76" smashed="yes">
+<attribute name="VALUE" x="-10.16" y="106.68" size="1.778" layer="96" rot="R90"/>
+</instance>
+<instance part="VSS42" gate="G$1" x="-10.16" y="149.86" smashed="yes">
+<attribute name="VALUE" x="-12.7" y="144.78" size="1.778" layer="96" rot="R90"/>
+</instance>
+<instance part="GND_POINTS" gate="G$1" x="53.34" y="152.4" smashed="yes">
+<attribute name="NAME" x="46.99" y="158.115" size="1.778" layer="95"/>
+<attribute name="VALUE" x="46.99" y="147.32" size="1.778" layer="96"/>
+</instance>
+<instance part="VSS43" gate="G$1" x="40.64" y="149.86" smashed="yes">
+<attribute name="VALUE" x="38.1" y="144.78" size="1.778" layer="96" rot="R90"/>
 </instance>
 </instances>
@@
 </segment>
 <segment>
-<wire x1="-22.86" y1="154.94" x2="-10.16" y2="154.94" width="0.1524" layer="91"/>
-<pinref part="JP3" gate="G$1" pin="1"/>
-<label x="-20.32" y="154.94" size="1.778" layer="95"/>
-<junction x="-22.86" y="154.94"/>
-</segment>
-<segment>
-<wire x1="-10.16" y1="124.46" x2="2.54" y2="124.46" width="0.1524" layer="91"/>
-<pinref part="JP4" gate="G$1" pin="1"/>
+<wire x1="-22.86" y1="162.56" x2="-10.16" y2="162.56" width="0.1524" layer="91"/>
+<label x="-27.94" y="165.1" size="1.778" layer="95"/>
+<junction x="-22.86" y="162.56"/>
+<pinref part="SJ2" gate="G$1" pin="1"/>
+<junction x="-10.16" y="162.56"/>
+</segment>
+<segment>
 <label x="-2.54" y="124.46" size="1.778" layer="95"/>
 <junction x="2.54" y="124.46"/>
+<pinref part="SJ1" gate="G$1" pin="1"/>
+<wire x1="-7.62" y1="124.46" x2="2.54" y2="124.46" width="0.1524" layer="91"/>
+<junction x="-7.62" y="124.46"/>
 </segment>
 <segment>
@@
 <pinref part="VSS40" gate="G$1" pin="VSS"/>
 </segment>
+<segment>
+<pinref part="SJ1" gate="G$1" pin="3"/>
+<pinref part="VSS41" gate="G$1" pin="VSS"/>
+<junction x="-7.62" y="114.3"/>
+</segment>
+<segment>
+<pinref part="SJ2" gate="G$1" pin="3"/>
+<pinref part="VSS42" gate="G$1" pin="VSS"/>
+<junction x="-10.16" y="152.4"/>
+</segment>
+<segment>
+<pinref part="GND_POINTS" gate="G$1" pin="2"/>
+<wire x1="50.8" y1="152.4" x2="40.64" y2="152.4" width="0.1524" layer="91"/>
+<wire x1="40.64" y1="152.4" x2="40.64" y2="154.94" width="0.1524" layer="91"/>
+<pinref part="GND_POINTS" gate="G$1" pin="1"/>
+<wire x1="40.64" y1="154.94" x2="50.8" y2="154.94" width="0.1524" layer="91"/>
+<pinref part="VSS43" gate="G$1" pin="VSS"/>
+<junction x="40.64" y="152.4"/>
+<junction x="50.8" y="152.4"/>
+<junction x="50.8" y="154.94"/>
+</segment>
 </net>
 <net name="AVDD" class="2">
@@
 <pinref part="IC2" gate="G$1" pin="SHDN"/>
 <wire x1="-25.4" y1="134.62" x2="-20.32" y2="134.62" width="0.1524" layer="91"/>
-<wire x1="-20.32" y1="134.62" x2="-20.32" y2="121.92" width="0.1524" layer="91"/>
-<pinref part="JP4" gate="G$1" pin="2"/>
-<wire x1="-20.32" y1="121.92" x2="-10.16" y2="121.92" width="0.1524" layer="91"/>
+<wire x1="-20.32" y1="134.62" x2="-20.32" y2="119.38" width="0.1524" layer="91"/>
 <junction x="-25.4" y="134.62"/>
+<pinref part="SJ1" gate="G$1" pin="2"/>
+<wire x1="-20.32" y1="119.38" x2="-12.7" y2="119.38" width="0.1524" layer="91"/>
+<junction x="-12.7" y="119.38"/>
 </segment>
 </net>
@@
 <pinref part="IC2" gate="G$1" pin="S"/>
 <wire x1="-25.4" y1="142.24" x2="-20.32" y2="142.24" width="0.1524" layer="91"/>
-<wire x1="-20.32" y1="142.24" x2="-20.32" y2="152.4" width="0.1524" layer="91"/>
-<pinref part="JP3" gate="G$1" pin="2"/>
-<wire x1="-20.32" y1="152.4" x2="-10.16" y2="152.4" width="0.1524" layer="91"/>
+<wire x1="-20.32" y1="142.24" x2="-20.32" y2="157.48" width="0.1524" layer="91"/>
 <junction x="-25.4" y="142.24"/>
-</segment>
-</net>
+<pinref part="SJ2" gate="G$1" pin="2"/>
+<wire x1="-20.32" y1="157.48" x2="-15.24" y2="157.48" width="0.1524" layer="91"/>
+<junction x="-15.24" y="157.48"/>
+</segment>
+</net>
