File: btob.brd (EAGLE design)
At the start: 107.9 x 8.6 mm, 4 parts, among them J1 MLE-105-01-G-DV, J2 MLE-105-01-G-DV, J3 MLE-105-01-G-DV

Commit message: rework for small sensor board with SCL imu chip
Connections:
- net N$1 renamed PIN9
- net N$10 renamed PIN2
- net N$2 renamed PIN7
- net N$3 renamed PIN5
- net N$4 renamed PIN3
- net N$5 renamed PIN1
- net N$6 renamed PIN10
- net N$7 renamed PIN8
- net N$8 renamed PIN6
- net N$9 renamed PIN4
Changed lines of the file:
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@@
 </elements>
 <signals>
-<signal name="N$1">
+<signal name="PIN9">
 <contactref element="J1" pad="9"/>
 <contactref element="SV1" pad="9"/>
@@
 <via x="51.3588" y="92.964" extent="1-16" drill="0.35"/>
 </signal>
-<signal name="N$2">
+<signal name="PIN7">
 <contactref element="J1" pad="7"/>
 <contactref element="SV1" pad="7"/>
@@
 <via x="50.7492" y="94.1832" extent="1-16" drill="0.35"/>
 </signal>
-<signal name="N$3">
+<signal name="PIN5">
 <contactref element="J1" pad="5"/>
 <contactref element="SV1" pad="5"/>
@@
 <via x="65.8368" y="93.4212" extent="1-16" drill="0.35"/>
 </signal>
-<signal name="N$4">
+<signal name="PIN3">
 <contactref element="J1" pad="3"/>
 <contactref element="SV1" pad="3"/>
@@
 <via x="60.3504" y="91.7448" extent="1-16" drill="0.35"/>
 </signal>
-<signal name="N$5">
+<signal name="PIN1">
 <contactref element="J1" pad="1"/>
 <contactref element="SV1" pad="1"/>
@@
 <via x="58.3692" y="92.964" extent="1-16" drill="0.35"/>
 </signal>
-<signal name="N$6">
+<signal name="PIN10">
 <contactref element="J1" pad="10"/>
 <contactref element="SV1" pad="10"/>
@@
 <via x="51.6636" y="89.6112" extent="1-16" drill="0.35"/>
 </signal>
-<signal name="N$7">
+<signal name="PIN8">
 <contactref element="J1" pad="8"/>
 <contactref element="SV1" pad="8"/>
@@
 <via x="51.6636" y="94.1832" extent="1-16" drill="0.35"/>
 </signal>
-<signal name="N$8">
+<signal name="PIN6">
 <contactref element="J1" pad="6"/>
 <contactref element="SV1" pad="6"/>
@@
 <via x="59.5884" y="92.3544" extent="1-16" drill="0.35"/>
 </signal>
-<signal name="N$9">
+<signal name="PIN4">
 <contactref element="J1" pad="4"/>
 <contactref element="SV1" pad="4"/>
@@
 <via x="60.3504" y="92.964" extent="1-16" drill="0.35"/>
 </signal>
-<signal name="N$10">
+<signal name="PIN2">
 <contactref element="J1" pad="2"/>
 <contactref element="SV1" pad="2"/>
