File: btob.sch (EAGLE design)
At the start: 4 parts, among them J1 MLE-105-01-G-DV, J2 MLE-105-01-G-DV, J3 MLE-105-01-G-DV

Commit message: up
Connections:
- net N$1 renamed P9
- net N$10 renamed P2
- net N$2 renamed P7
- net N$3 renamed P5
- net N$4 renamed P3
- net N$5 renamed P1
- net N$6 renamed P10
- net N$7 renamed P8
- net N$8 renamed P6
- net N$9 renamed P4
Changed lines of the file:
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@@
 </busses>
 <nets>
-<net name="N$1" class="0">
+<net name="P9" class="0">
 <segment>
 <pinref part="J1" gate="G$1" pin="9"/>
 <wire x1="17.78" y1="76.2" x2="7.62" y2="76.2" width="0.1524" layer="91"/>
+<label x="2.54" y="76.2" size="1.778" layer="95"/>
 </segment>
 <segment>
@@
 </segment>
 </net>
-<net name="N$2" class="0">
+<net name="P7" class="0">
 <segment>
 <pinref part="J1" gate="G$1" pin="7"/>
 <wire x1="17.78" y1="73.66" x2="7.62" y2="73.66" width="0.1524" layer="91"/>
+<label x="2.54" y="73.66" size="1.778" layer="95"/>
 </segment>
 <segment>
@@
 </segment>
 </net>
-<net name="N$3" class="0">
+<net name="P5" class="0">
 <segment>
 <pinref part="J1" gate="G$1" pin="5"/>
 <wire x1="17.78" y1="71.12" x2="7.62" y2="71.12" width="0.1524" layer="91"/>
+<label x="2.54" y="71.12" size="1.778" layer="95"/>
 </segment>
 <segment>
@@
 </segment>
 </net>
-<net name="N$4" class="0">
+<net name="P3" class="0">
 <segment>
 <pinref part="J1" gate="G$1" pin="3"/>
 <wire x1="17.78" y1="68.58" x2="7.62" y2="68.58" width="0.1524" layer="91"/>
+<label x="2.54" y="68.58" size="1.778" layer="95"/>
 </segment>
 <segment>
@@
 </segment>
 </net>
-<net name="N$5" class="0">
+<net name="P1" class="0">
 <segment>
 <pinref part="J1" gate="G$1" pin="1"/>
 <wire x1="17.78" y1="66.04" x2="7.62" y2="66.04" width="0.1524" layer="91"/>
+<label x="2.54" y="66.04" size="1.778" layer="95"/>
 </segment>
 <segment>
@@
 </segment>
 </net>
-<net name="N$6" class="0">
+<net name="P10" class="0">
 <segment>
 <pinref part="J1" gate="G$1" pin="10"/>
 <wire x1="40.64" y1="76.2" x2="55.88" y2="76.2" width="0.1524" layer="91"/>
+<label x="58.42" y="76.2" size="1.778" layer="95"/>
 </segment>
 <segment>
@@
 </segment>
 </net>
-<net name="N$7" class="0">
+<net name="P8" class="0">
 <segment>
 <pinref part="J1" gate="G$1" pin="8"/>
 <wire x1="40.64" y1="73.66" x2="55.88" y2="73.66" width="0.1524" layer="91"/>
+<label x="58.42" y="73.66" size="1.778" layer="95"/>
 </segment>
 <segment>
@@
 </segment>
 </net>
-<net name="N$8" class="0">
+<net name="P6" class="0">
 <segment>
 <pinref part="J1" gate="G$1" pin="6"/>
 <wire x1="40.64" y1="71.12" x2="55.88" y2="71.12" width="0.1524" layer="91"/>
+<label x="58.42" y="71.12" size="1.778" layer="95"/>
 </segment>
 <segment>
@@
 </segment>
 </net>
-<net name="N$9" class="0">
+<net name="P4" class="0">
 <segment>
 <pinref part="J1" gate="G$1" pin="4"/>
 <wire x1="40.64" y1="68.58" x2="55.88" y2="68.58" width="0.1524" layer="91"/>
+<label x="58.42" y="68.58" size="1.778" layer="95"/>
 </segment>
 <segment>
@@
 </segment>
 </net>
-<net name="N$10" class="0">
+<net name="P2" class="0">
 <segment>
 <pinref part="J1" gate="G$1" pin="2"/>
 <wire x1="40.64" y1="66.04" x2="55.88" y2="66.04" width="0.1524" layer="91"/>
+<label x="58.42" y="66.04" size="1.778" layer="95"/>
 </segment>
 <segment>
